File: hardware/PCB/dev_02_kicad/_autosave-Core1.kicad_pcb (KiCad board)
At the start: 2 copper layers, 50 x 43.6 mm, 28 parts, among them P1 USB_OTG, P2 JST PH Connector, P3 CONN_01X04, P4 Mic_IN, P5 MCP3201, P6 JST PH Connector, P7 USB_OTG, P8 CONN_01X04, SW1 SW_PUSH, U1 ESP-07v2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

Commit message: Inför träff
Alla ändringar inför träff
Parts:
- removed C1: C, Capacitors_SMD:C_0805
- C2: value C -> 0,1uF
- R1: value 333 -> 10k
- moved C6 12.8 mm to (156.8, 124.0), turned to 90 degrees
- moved C5 12.0 mm to (163.8, 124.0), turned to 90 degrees
- moved P4 2.81 mm to (135.0, 117.1)
- moved P5 2.39 mm to (130.4, 119.3)
- moved P6 2.39 mm to (121.7, 119.0)
- moved F1 2.01 mm to (160.3, 123.8), turned to 90 degrees
- moved P8 1.54 mm to (143.1, 119.8)
- moved P7 0.91 mm to (162.2, 115.1)
Connections:
- U1 pad 2: Net-(R1-Pad2) -> Net-(U1-Pad2)
- U1 pad 3: Net-(U1-Pad3) -> Net-(R1-Pad2)
Routing:
- net Net-(F1-Pad1): track 14.8 -> 23.7 mm
- net +5V: track 13.2 -> 21.0 mm
- net Net-(C5-Pad2): track 10.9 -> 17.0 mm
- net Net-(D1-Pad2): track 0.07 -> 3.19 mm
- net GNDA: track 99.3 -> 101.5 mm, vias 2 -> 3
- net Net-(R1-Pad2): track 12.3 -> 10.2 mm
- net RX_A: track 13.8 -> 12.1 mm
- net AnalogIn: track 7.44 -> 6.10 mm
- net TX_A: track 17.3 -> 16.2 mm
- net GNDD: track 35.7 -> 34.6 mm
Other:
- outline, holes or cut-outs redrawn
