File: hardware/PCB/dev_02_kicad/_saved_Core1.sch (KiCad schematic (older format))
At the start: 26 parts, among them P1 USB_OTG, P2 JST PH Connector, P3 CONN_01X04, P4 Mic_IN, P5 MCP3201, P6 JST PH Connector, P7 USB_OTG, P8 CONN_01X04, SW1 SW_PUSH, U1 ESP-07v2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

Commit message: Inför träff
Alla ändringar inför träff
Parts:
- removed C1: C, Capacitors_SMD:C_0805, symbol C
- C2: value C -> 0,1uF
- R1: value 333 -> 10k
Connections:
- net at U1.2 (ADC): no longer R1.2
- net at U1.3 (CH_PD): now also R1.2
Other:
- note added: "Digikey; \nMCP3201T-CI/SNDKR-ND"
Changed lines of the file:
@@
 P 1450 3200
 F 0 "C2" H 1475 3300 50  0000 L CNN
-F 1 "C" H 1475 3100 50  0000 L CNN
+F 1 "0,1uF" H 1475 3100 50  0000 L CNN
 F 2 "Capacitors_SMD:C_0805" H 1488 3050 50  0001 C CNN
 F 3 "" H 1450 3200 50  0000 C CNN
 	1    1450 3200
-	0    1    1    0
-$EndComp
-$Comp
-L C C1
-U 1 1 57F1559F
-P 1450 3000
-F 0 "C1" H 1475 3100 50  0000 L CNN
-F 1 "C" H 1475 2900 50  0000 L CNN
-F 2 "Capacitors_SMD:C_0805" H 1488 2850 50  0001 C CNN
-F 3 "" H 1450 3000 50  0000 C CNN
-	1    1450 3000
 	0    1    1    0
 $EndComp
@@
 $EndComp
 $Comp
-L GND #PWR03
-U 1 1 57F156AD
-P 1150 3000
-F 0 "#PWR03" H 1150 2750 50  0001 C CNN
-F 1 "GND" H 1150 2850 50  0000 C CNN
-F 2 "" H 1150 3000 50  0000 C CNN
-F 3 "" H 1150 3000 50  0000 C CNN
-	1    1150 3000
-	0    1    -1   0
-$EndComp
-$Comp
 L +5V #PWR04
 U 1 1 57F15791
@@
 P 1600 1800
 F 0 "R1" V 1680 1800 50  0000 C CNN
-F 1 "333" V 1600 1800 50  0000 C CNN
+F 1 "10k" V 1600 1800 50  0000 C CNN
 F 2 "Resistors_SMD:R_0805" V 1530 1800 50  0001 C CNN
 F 3 "" H 1600 1800 50  0000 C CNN
@@
 NoConn ~ 3700 2000
 NoConn ~ 1900 1700
-NoConn ~ 1900 1900
 NoConn ~ 1900 2000
 NoConn ~ 1900 2300
@@
 L GNDA #PWR019
 U 1 1 57F44280
-P 7900 4050
-F 0 "#PWR019" H 7900 3800 50  0001 C CNN
-F 1 "GNDA" H 7900 3900 50  0000 C CNN
-F 2 "" H 7900 4050 50  0000 C CNN
-F 3 "" H 7900 4050 50  0000 C CNN
-	1    7900 4050
+P 7800 3900
+F 0 "#PWR019" H 7800 3650 50  0001 C CNN
+F 1 "GNDA" H 7800 3750 50  0000 C CNN
+F 2 "" H 7800 3900 50  0000 C CNN
+F 3 "" H 7800 3900 50  0000 C CNN
+	1    7800 3900
 	0    -1   -1   0
 $EndComp
@@
 	1750 3200 1600 3200
 Wire Wire Line
-	1600 3000 1750 3000
-Wire Wire Line
-	1300 3000 1150 3000
-Wire Wire Line
 	1150 3200 1300 3200
 Wire Wire Line
 	2400 4300 1750 4300
 Connection ~ 1750 4300
-Wire Wire Line
-	1900 1800 1750 1800
 Wire Wire Line
 	1250 1800 1450 1800
@@
 	7650 3900 7800 3900
 Wire Wire Line
-	7800 3900 7800 4200
-Wire Wire Line
 	7800 4200 7650 4200
-Wire Wire Line
-	7800 4050 7900 4050
-Connection ~ 7800 4050
 Wire Bus Line
 	6100 5050 550  5050
@@
 $EndComp
 NoConn ~ 7000 4700
+$Comp
+L GNDA #PWR?
+U 1 1 57F5436B
+P 7800 4200
+F 0 "#PWR?" H 7800 3950 50  0001 C CNN
+F 1 "GNDA" H 7800 4050 50  0000 C CNN
+F 2 "" H 7800 4200 50  0000 C CNN
+F 3 "" H 7800 4200 50  0000 C CNN
+	1    7800 4200
+	0    -1   -1   0
+$EndComp
+Text Notes 1800 5400 0    60   ~ 0
+Digikey; \nMCP3201T-CI/SNDKR-ND
+Wire Wire Line
+	1750 1800 1750 1900
+Wire Wire Line
+	1750 1900 1900 1900
+NoConn ~ 1900 1800
 $EndSCHEMATC
