File: hardware/PCB/dev_02_kicad/Core1.kicad_pcb (KiCad board)
At the start: 2 copper layers, 50 x 43.6 mm, 28 parts, among them P1 USB_OTG, P2 JST PH Connector, P3 CONN_01X04, P4 Mic_IN, P5 MCP3201, P6 JST PH Connector, P7 USB_OTG, P8 CONN_01X04, SW1 SW_PUSH, U1 ESP-07v2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

Commit message: Ljudet fungerar!
Ljud fungerar-
Parts:
- removed C1: C, Capacitors_SMD:C_0805
- removed REF** (x2): 1pin, Connect:1pin
- added ?: , Mounting_Holes:MountingHole_2.5mm, F.Cu at (162.5, 87.1)
- added ?: , Mounting_Holes:MountingHole_2.5mm, F.Cu at (119.6, 105.1)
- C2: value C -> 0,1uF
- P2: value JST PH Connector -> Pinhead SMD Connector; footprint Connectors_JST:JST_PH_S5B-PH-SM4-TB_05x2.00mm_Angled -> KiCad libraries:Pin_Header_Angled_1x05_SMD
- P6: value JST PH Connector -> AudioConnector; footprint Connectors_JST:JST_PH_S5B-PH-SM4-TB_05x2.00mm_Angled -> KiCad libraries:Pin_Header_Angled_1x05_SMD
- R1: value 333 -> 10k
- moved C6 12.8 mm to (156.8, 124.0), turned to 90 degrees
- moved C5 12.0 mm to (163.8, 124.0), turned to 90 degrees
- moved P6 8.13 mm to (125.4, 124.0), turned to 180 degrees
- moved P4 7.35 mm to (135.7, 122.0), turned to 180 degrees
- moved P2 6.33 mm to (144.2, 93.6), turned to 90 degrees
- moved P5 2.39 mm to (130.4, 119.3)
- moved F1 1.93 mm to (160.3, 124.4), turned to 90 degrees
- moved P8 1.54 mm to (143.1, 119.8)
- moved SW1 0.73 mm to (151.2, 100.2)
- moved P7 0.51 mm to (162.2, 115.5)
Connections:
- P1 pad 2: Net-(P1-Pad2) -> (no net)
- P1 pad 3: Net-(P1-Pad3) -> (no net)
- P1 pad 4: Net-(P1-Pad4) -> (no net)
- P2 pad 1: +3V3 -> GND
- P2 pad 2: SS -> SCLK
- P2 pad 4: SCLK -> SS
- P2 pad 5: GND -> +3V3
- P6 pad 1: VCC_A -> GNDD
- P6 pad 2: SS_A -> SCLK_A
- P6 pad 4: SCLK_A -> SS_A
- P6 pad 5: GNDD -> VCC_A
- P7 pad 4: Net-(P7-Pad4) -> (no net)
- U1 pad 1: Net-(U1-Pad1) -> (no net)
- U1 pad 13: Net-(U1-Pad13) -> (no net)
- U1 pad 2: Net-(R1-Pad2) -> (no net)
- U1 pad 3: Net-(U1-Pad3) -> Net-(R1-Pad2)
- U1 pad 4: Net-(U1-Pad4) -> (no net)
- U1 pad 7: Net-(U1-Pad7) -> (no net)
- U3 pad 10: Net-(U3-Pad10) -> (no net)
- U3 pad 11: Net-(U3-Pad11) -> (no net)
- U3 pad 12: Net-(U3-Pad12) -> (no net)
- U3 pad 13: Net-(U3-Pad13) -> (no net)
- U3 pad 14: Net-(U3-Pad14) -> (no net)
- U3 pad 17: Net-(U3-Pad17) -> (no net)
- U3 pad 19: Net-(U3-Pad19) -> (no net)
- U3 pad 2: Net-(U3-Pad2) -> (no net)
- U3 pad 27: Net-(U3-Pad27) -> (no net)
- U3 pad 28: Net-(U3-Pad28) -> (no net)
- U3 pad 3: Net-(U3-Pad3) -> (no net)
- U3 pad 6: Net-(U3-Pad6) -> (no net)
- U3 pad 9: Net-(U3-Pad9) -> (no net)
Routing:
- net GND: track 120.3 -> 132.9 mm, vias 0 -> 2
- net Net-(F1-Pad1): track 14.8 -> 27.0 mm
- net +5V: track 13.2 -> 21.0 mm
- net AnalogIn: track 7.44 -> 12.2 mm
- net Net-(C5-Pad2): track 10.9 -> 14.9 mm
- net GNDA: track 99.3 -> 95.9 mm, vias 2 -> 4
- net Net-(D1-Pad2): track 0.07 -> 3.19 mm
- net Net-(R1-Pad2): track 12.3 -> 10.2 mm
- net SCLK: track 22.9 -> 20.9 mm
- net RX_A: track 13.8 -> 12.1 mm
- net VCC_A: track 33.3 -> 34.9 mm, vias 1 -> 0
- net SS_A: track 4.17 -> 5.52 mm
- net MISO: track 22.8 -> 21.5 mm
- net TX_A: track 17.3 -> 16.2 mm
- net SS: track 21.5 -> 22.4 mm
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Other:
- outline, holes or cut-outs redrawn
- rule trace_min: 0.2 -> 0.3
