File: hardware/PCB/dev_02_kicad/Core1.sch (KiCad schematic (older format))
At the start: 14 parts, among them P1 USB_OTG, P2 JST PH Connector, P3 CONN_01X04, SW1 SW_PUSH, U1 ESP-07v2, U2 LM1117-3.3

Commit message: Inför träff
Alla ändringar inför träff
Parts:
- added C5, C6: C, Capacitors_SMD:C_0805, symbol C
- added D1, D2: LED, LEDs:LED_0805, symbol LED
- added P4: Mic_IN, Pin_Headers:Pin_Header_Straight_1x03, symbol CONN_01X03
- added P5: MCP3201, Housings_SOIC:SOIC-8_3.9x4.9mm_Pitch1.27mm, symbol CONN_02X04
- added P6: JST PH Connector, Connectors_JST:JST_PH_S5B-PH-SM4-TB_05x2.00mm_Angled, symbol CONN_01X05
- added P7: USB_OTG, Connect:USB_Mini-B, symbol USB_OTG
- added P8: CONN_01X04, Pin_Headers:Pin_Header_Straight_1x04, symbol CONN_01X04
- added R4, R5: 333, Resistors_SMD:R_0805, symbol R
- added U3: FT232RL, Housings_SSOP:SSOP-28_5.3x10.2mm_Pitch0.65mm, symbol FT232RL
Connections:
- net +5V: now also P1.1 (VCC); no longer F1.1
- net at F1.2: now also C5.2, C6.2, P7.1 (VCC); no longer P1.1 (VCC)
- new net: F1.1, U3.20 (VCC)
- new net: D1.1 (K), U3.22 (CBUS1)
- new net: D2.1 (K), U3.23 (CBUS0)
- new net: D1.2 (A), R4.1
- new net: D2.2 (A), R5.1
- new net AnalogIn: P4.3 (P3), P5.3 (P3)
- new net GNDA: C5.1, C6.1, P7.5 (GND), P7.6 (shield), P8.1 (P1), P8.4 (P4), U3.18 (GND), U3.21 (GND), U3.25 (AGND), U3.26 (TEST), U3.7 (GND)
- new net GNDD: P4.2 (P2), P5.5 (P5), P5.7 (P7), P6.5 (P5)
- new net MISO_A: P5.6 (P6), P6.3 (P3)
- new net RX_A: P8.2 (P2), U3.5 (RXD)
- new net SCLK_A: P5.4 (P4), P6.4 (P4)
- new net SS_A: P5.8 (P8), P6.2 (P2)
- new net TX_A: P8.3 (P3), U3.1 (TXD)
- new net USBDm: P7.2 (D-), U3.16 (USBDM)
- new net USBDp: P7.3 (D+), U3.15 (USBDP)
- new net VCCIO: R4.2, R5.2, U3.4 (VCCIO)
- new net VCC_A: P4.1 (P1), P5.1 (P1), P5.2 (P2), P6.1 (P1)
- no-connect marks 6 -> 22
Other:
- note added: "Hold for Wifi settings reset"
- moved on the sheet: C1, C2, C3, C4, F1, P1, P2, P3, R1, R2, R3, SW1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

Commit message: Ljudet fungerar!
Ljud fungerar-
Parts:
- removed C1: C, Capacitors_SMD:C_0805, symbol C
- C2: value C -> 0,1uF
- P2, P6: value JST PH Connector -> Pinhead SMD Connector; footprint Connectors_JST:JST_PH_S5B-PH-SM4-TB_05x2.00mm_Angled -> KiCad libraries:Pin_Header_Angled_1x05_SMD
- R1: value 333 -> 10k
Connections:
- net +3V3: now also P2.5 (P5); no longer P2.1 (P1)
- net GND: now also P2.1 (P1); no longer P2.5 (P5)
- net GNDD: now also P6.1 (P1); no longer P6.5 (P5)
- net SCLK: now also P2.2 (P2); no longer P2.4 (P4)
- net SCLK_A: now also P6.2 (P2); no longer P6.4 (P4)
- net SS: now also P2.4 (P4); no longer P2.2 (P2)
- net SS_A: now also P6.4 (P4); no longer P6.2 (P2)
- net VCC_A: now also P6.5 (P5); no longer P6.1 (P1)
- net at U1.2 (ADC): no longer R1.2
- net at U1.3 (CH_PD): now also R1.2
Other:
- note added: "Digikey; \nMCP3201T-CI/SNDKR-ND"
- note added: "http://www.digikey.com/product-search/en/connectors-interconnects/rectangular-connectors-headers-male-pins/1442547?k=header&k=&pkeyword=header&v=19&FV=1140160%2C1600018%2C1600309%2C160045f%2C8000010%2Cfff40016%2Cfff802f3&mnonly=0&newproducts=0&ColumnSort=0&page=1&quantity=0&ptm=0&fid=0&pageSize=25"
Changed lines of the file:
@@
 LIBS:mm232r
 LIBS:ft232rl
+LIBS:SundbergKiCadLib
 LIBS:Core1-cache
 EELAYER 25 0
@@
 P 1450 3200
 F 0 "C2" H 1475 3300 50  0000 L CNN
-F 1 "C" H 1475 3100 50  0000 L CNN
+F 1 "0,1uF" H 1475 3100 50  0000 L CNN
 F 2 "Capacitors_SMD:C_0805" H 1488 3050 50  0001 C CNN
 F 3 "" H 1450 3200 50  0000 C CNN
 	1    1450 3200
-	0    1    1    0
-$EndComp
-$Comp
-L C C1
-U 1 1 57F1559F
-P 1450 3000
-F 0 "C1" H 1475 3100 50  0000 L CNN
-F 1 "C" H 1475 2900 50  0000 L CNN
-F 2 "Capacitors_SMD:C_0805" H 1488 2850 50  0001 C CNN
-F 3 "" H 1450 3000 50  0000 C CNN
-	1    1450 3000
 	0    1    1    0
 $EndComp
@@
 $EndComp
 $Comp
-L GND #PWR03
-U 1 1 57F156AD
-P 1150 3000
-F 0 "#PWR03" H 1150 2750 50  0001 C CNN
-F 1 "GND" H 1150 2850 50  0000 C CNN
-F 2 "" H 1150 3000 50  0000 C CNN
-F 3 "" H 1150 3000 50  0000 C CNN
-	1    1150 3000
-	0    1    -1   0
-$EndComp
-$Comp
-L +5V #PWR04
+L +5V #PWR03
 U 1 1 57F15791
 P 1750 2800
-F 0 "#PWR04" H 1750 2650 50  0001 C CNN
+F 0 "#PWR03" H 1750 2650 50  0001 C CNN
 F 1 "+5V" H 1750 2940 50  0000 C CNN
 F 2 "" H 1750 2800 50  0000 C CNN
@@
 P 1600 1800
 F 0 "R1" V 1680 1800 50  0000 C CNN
-F 1 "333" V 1600 1800 50  0000 C CNN
+F 1 "10k" V 1600 1800 50  0000 C CNN
 F 2 "Resistors_SMD:R_0805" V 1530 1800 50  0001 C CNN
 F 3 "" H 1600 1800 50  0000 C CNN
@@
 $EndComp
 $Comp
-L +3V3 #PWR05
+L +3V3 #PWR04
 U 1 1 57F166B6
 P 1250 1800
-F 0 "#PWR05" H 1250 1650 50  0001 C CNN
+F 0 "#PWR04" H 1250 1650 50  0001 C CNN
 F 1 "+3V3" H 1250 1940 50  0000 C CNN
 F 2 "" H 1250 1800 50  0000 C CNN
@@
 $EndComp
 $Comp
-L GND #PWR06
+L GND #PWR05
 U 1 1 57F16885
 P 3900 2900
-F 0 "#PWR06" H 3900 2650 50  0001 C CNN
+F 0 "#PWR05" H 3900 2650 50  0001 C CNN
 F 1 "GND" H 3900 2750 50  0000 C CNN
 F 2 "" H 3900 2900 50  0000 C CNN
@@
 SS
 $Comp
-L GND #PWR07
+L GND #PWR06
 U 1 1 57F16C4F
 P 5600 1900
-F 0 "#PWR07" H 5600 1650 50  0001 C CNN
+F 0 "#PWR06" H 5600 1650 50  0001 C CNN
 F 1 "GND" H 5600 1750 50  0000 C CNN
 F 2 "" H 5600 1900 50  0000 C CNN
@@
 $EndComp
 $Comp
-L +5V #PWR08
+L +5V #PWR07
 U 1 1 57F18D71
 P 3150 3600
-F 0 "#PWR08" H 3150 3450 50  0001 C CNN
+F 0 "#PWR07" H 3150 3450 50  0001 C CNN
 F 1 "+5V" H 3150 3740 50  0000 C CNN
 F 2 "" H 3150 3600 50  0000 C CNN
@@
 $EndComp
 $Comp
-L GND #PWR09
+L GND #PWR08
 U 1 1 57F18E7E
 P 3850 4150
-F 0 "#PWR09" H 3850 3900 50  0001 C CNN
+F 0 "#PWR08" H 3850 3900 50  0001 C CNN
 F 1 "GND" H 3850 4000 50  0000 C CNN
 F 2 "" H 3850 4150 50  0000 C CNN
@@
 $EndComp
 $Comp
-L +3V3 #PWR010
+L +3V3 #PWR09
 U 1 1 57F18EBF
 P 4550 3600
-F 0 "#PWR010" H 4550 3450 50  0001 C CNN
+F 0 "#PWR09" H 4550 3450 50  0001 C CNN
 F 1 "+3V3" H 4550 3740 50  0000 C CNN
 F 2 "" H 4550 3600 50  0000 C CNN
@@
 P 5350 3050
 F 0 "P2" H 5350 3350 50  0000 C CNN
-F 1 "JST PH Connector" V 5450 3050 50  0000 C CNN
-F 2 "Connectors_JST:JST_PH_S5B-PH-SM4-TB_05x2.00mm_Angled" H 5350 3050 50  0001 C CNN
+F 1 "Pinhead SMD Connector" V 5450 3050 50  0000 C CNN
+F 2 "KiCad libraries:Pin_Header_Angled_1x05_SMD" H 5350 3050 50  0001 C CNN
 F 3 "" H 5350 3050 50  0000 C CNN
 	1    5350 3050
@@
 $EndComp
 $Comp
-L GND #PWR011
+L GND #PWR010
 U 1 1 57F1ABC7
+P 5550 2750
+F 0 "#PWR010" H 5550 2500 50  0001 C CNN
+F 1 "GND" H 5550 2600 50  0000 C CNN
+F 2 "" H 5550 2750 50  0000 C CNN
+F 3 "" H 5550 2750 50  0000 C CNN
+	1    5550 2750
+	-1   0    0    1
+$EndComp
+$Comp
+L +3V3 #PWR011
+U 1 1 57F1ADAD
 P 5150 2750
-F 0 "#PWR011" H 5150 2500 50  0001 C CNN
-F 1 "GND" H 5150 2600 50  0000 C CNN
+F 0 "#PWR011" H 5150 2600 50  0001 C CNN
+F 1 "+3V3" H 5150 2890 50  0000 C CNN
 F 2 "" H 5150 2750 50  0000 C CNN
 F 3 "" H 5150 2750 50  0000 C CNN
 	1    5150 2750
-	-1   0    0    1
-$EndComp
-$Comp
-L +3V3 #PWR012
-U 1 1 57F1ADAD
-P 5550 2750
-F 0 "#PWR012" H 5550 2600 50  0001 C CNN
-F 1 "+3V3" H 5550 2890 50  0000 C CNN
-F 2 "" H 5550 2750 50  0000 C CNN
-F 3 "" H 5550 2750 50  0000 C CNN
-	1    5550 2750
-	1    0    0    -1
-$EndComp
-Text GLabel 5250 2750 1    60   Input ~ 0
+	1    0    0    -1
+$EndComp
+Text GLabel 5450 2750 1    60   Input ~ 0
 SCLK
 Text GLabel 5350 2750 1    60   Input ~ 0
 MISO
-Text GLabel 5450 2750 1    60   Input ~ 0
+Text GLabel 5250 2750 1    60   Input ~ 0
 SS
 NoConn ~ 3700 2000
 NoConn ~ 1900 1700
-NoConn ~ 1900 1900
 NoConn ~ 1900 2000
 NoConn ~ 1900 2300
 NoConn ~ 2000 4000
 $Comp
-L +3V3 #PWR013
+L +3V3 #PWR012
 U 1 1 57F1C007
 P 5150 1700
-F 0 "#PWR013" H 5150 1550 50  0001 C CNN
+F 0 "#PWR012" H 5150 1550 50  0001 C CNN
 F 1 "+3V3" H 5150 1840 50  0000 C CNN
 F 2 "" H 5150 1700 50  0000 C CNN
@@
 $EndComp
 $Comp
-L GND #PWR014
+L GND #PWR013
 U 1 1 57F1DA9B
 P 4300 4050
-F 0 "#PWR014" H 4300 3800 50  0001 C CNN
+F 0 "#PWR013" H 4300 3800 50  0001 C CNN
 F 1 "GND" H 4300 3900 50  0000 C CNN
 F 2 "" H 4300 4050 50  0000 C CNN
@@
 $EndComp
 $Comp
-L GND #PWR015
+L GND #PWR014
 U 1 1 57F1DADF
 P 3400 4050
-F 0 "#PWR015" H 3400 3800 50  0001 C CNN
+F 0 "#PWR014" H 3400 3800 50  0001 C CNN
 F 1 "GND" H 3400 3900 50  0000 C CNN
 F 2 "" H 3400 4050 50  0000 C CNN
@@
 Digikey: 455-1752-6-ND
 $Comp
-L GND #PWR016
+L GND #PWR015
 U 1 1 57F3D7C8
 P 4450 1200
-F 0 "#PWR016" H 4450 950 50  0001 C CNN
+F 0 "#PWR015" H 4450 950 50  0001 C CNN
 F 1 "GND" H 4450 1050 50  0000 C CNN
 F 2 "" H 4450 1200 50  0000 C CNN
@@
 USBDm
 $Comp
-L GNDA #PWR017
+L GNDA #PWR016
 U 1 1 57F4214D
 P 6550 4500
-F 0 "#PWR017" H 6550 4250 50  0001 C CNN
+F 0 "#PWR016" H 6550 4250 50  0001 C CNN
 F 1 "GNDA" H 6550 4350 50  0000 C CNN
 F 2 "" H 6550 4500 50  0000 C CNN
@@
 $EndComp
 $Comp
-L GNDA #PWR018
+L GNDA #PWR017
 U 1 1 57F426AC
 P 9300 4800
-F 0 "#PWR018" H 9300 4550 50  0001 C CNN
+F 0 "#PWR017" H 9300 4550 50  0001 C CNN
 F 1 "GNDA" H 9300 4650 50  0000 C CNN
 F 2 "" H 9300 4800 50  0000 C CNN
@@
 VCCIO
 $Comp
-L GNDA #PWR019
+L GNDA #PWR018
 U 1 1 57F44280
 P 7800 3900
-F 0 "#PWR019" H 7800 3650 50  0001 C CNN
+F 0 "#PWR018" H 7800 3650 50  0001 C CNN
 F 1 "GNDA" H 7800 3750 50  0000 C CNN
 F 2 "" H 7800 3900 50  0000 C CNN
@@
 P 3100 7100
 F 0 "P6" H 3100 7400 50  0000 C CNN
-F 1 "JST PH Connector" V 3200 7100 50  0000 C CNN
-F 2 "Connectors_JST:JST_PH_S5B-PH-SM4-TB_05x2.00mm_Angled" H 3100 7100 50  0001 C CNN
+F 1 "Pinhead SMD Connector" V 3200 7100 50  0000 C CNN
+F 2 "KiCad libraries:Pin_Header_Angled_1x05_SMD" H 3100 7100 50  0001 C CNN
 F 3 "" H 3100 7100 50  0000 C CNN
 	1    3100 7100
@@
 VCC_A
 $Comp
-L GNDD #PWR020
+L GNDD #PWR019
 U 1 1 57F4646F
 P 1700 6150
-F 0 "#PWR020" H 1700 5900 50  0001 C CNN
+F 0 "#PWR019" H 1700 5900 50  0001 C CNN
 F 1 "GNDD" H 1700 6000 50  0000 C CNN
 F 2 "" H 1700 6150 50  0000 C CNN
@@
 $EndComp
 $Comp
-L GNDD #PWR021
+L GNDD #PWR020
 U 1 1 57F46607
 P 1150 6600
-F 0 "#PWR021" H 1150 6350 50  0001 C CNN
+F 0 "#PWR020" H 1150 6350 50  0001 C CNN
 F 1 "GNDD" H 1150 6450 50  0000 C CNN
 F 2 "" H 1150 6600 50  0000 C CNN
@@
 	1750 3200 1600 3200
 Wire Wire Line
-	1600 3000 1750 3000
-Wire Wire Line
-	1300 3000 1150 3000
-Wire Wire Line
 	1150 3200 1300 3200
 Wire Wire Line
 	2400 4300 1750 4300
 Connection ~ 1750 4300
-Wire Wire Line
-	1900 1800 1750 1800
 Wire Wire Line
 	1250 1800 1450 1800
@@
 Text GLabel 1250 7100 1    60   Input ~ 0
 VCC_A
-Text GLabel 2900 6900 0    60   Input ~ 0
+Text GLabel 2900 7300 0    60   Input ~ 0
 VCC_A
 Wire Wire Line
@@
 Wire Wire Line
 	2900 7200 2450 7200
-Text GLabel 2450 7200 0    60   Input ~ 0
+Text GLabel 2450 7000 0    60   Input ~ 0
 SCLK_A
 Text GLabel 2900 7100 0    60   Input ~ 0
 MISO_A
-Text GLabel 2450 7000 0    60   Input ~ 0
+Text GLabel 2450 7200 0    60   Input ~ 0
 SS_A
 $Comp
-L GNDD #PWR022
+L GNDD #PWR021
 U 1 1 57F481AC
-P 2900 7300
-F 0 "#PWR022" H 2900 7050 50  0001 C CNN
-F 1 "GNDD" H 2900 7150 50  0000 C CNN
-F 2 "" H 2900 7300 50  0000 C CNN
-F 3 "" H 2900 7300 50  0000 C CNN
-	1    2900 7300
+P 2900 6900
+F 0 "#PWR021" H 2900 6650 50  0001 C CNN
+F 1 "GNDD" H 2900 6750 50  0000 C CNN
+F 2 "" H 2900 6900 50  0000 C CNN
+F 3 "" H 2900 6900 50  0000 C CNN
+	1    2900 6900
 	0    1    1    0
 $EndComp
@@
 Connection ~ 9000 4050
 $Comp
-L GNDA #PWR023
+L GNDA #PWR022
 U 1 1 57F4A9AD
 P 9000 4200
-F 0 "#PWR023" H 9000 3950 50  0001 C CNN
+F 0 "#PWR022" H 9000 3950 50  0001 C CNN
 F 1 "GNDA" H 9000 4050 50  0000 C CNN
 F 2 "" H 9000 4200 50  0000 C CNN
@@
 NoConn ~ 7000 4700
 $Comp
-L GNDA #PWR?
+L GNDA #PWR023
 U 1 1 57F5436B
 P 7800 4200
-F 0 "#PWR?" H 7800 3950 50  0001 C CNN
+F 0 "#PWR023" H 7800 3950 50  0001 C CNN
 F 1 "GNDA" H 7800 4050 50  0000 C CNN
 F 2 "" H 7800 4200 50  0000 C CNN
@@
 	0    -1   -1   0
 $EndComp
+Text Notes 1800 5400 0    60   ~ 0
+Digikey; \nMCP3201T-CI/SNDKR-ND
+Wire Wire Line
+	1750 1800 1750 1900
+Wire Wire Line
+	1750 1900 1900 1900
+NoConn ~ 1900 1800
+Text Notes 3050 7550 0    60   ~ 0
+http://www.digikey.com/product-search/en/connectors-interconnects/rectangular-connectors-headers-male-pins/1442547?k=header&k=&pkeyword=header&v=19&FV=1140160%2C1600018%2C1600309%2C160045f%2C8000010%2Cfff40016%2Cfff802f3&mnonly=0&newproducts=0&ColumnSort=0&page=1&quantity=0&ptm=0&fid=0&pageSize=25
 $EndSCHEMATC
