File: hardware/PCB/dev_02_kicad/Core1.sch (KiCad schematic (older format))
At the start: 25 parts, among them P1 USB_OTG, P2 Pinhead SMD Connector, P3 CONN_01X04, P4 Mic_IN, P5 MCP3201, P6 Pinhead SMD Connector, P7 USB_OTG, P8 CONN_01X04, SW1 SW_PUSH, U1 ESP-07v2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

Commit message: UDPServer
Hela UDP Server projecktet
Connections:
- net SS: now also R2.1
- net at U1.11 (GPIO2): no longer R2.1
- no-connect marks 22 -> 23
Changed lines of the file:
@@
 LIBS:mm232r
 LIBS:ft232rl
+LIBS:Core1-cache
 EELAYER 25 0
 EELAYER END
@@
 Wire Wire Line
 	3700 2300 3850 2300
-Wire Wire Line
-	3700 2200 3750 2200
 Connection ~ 3750 2900
-Wire Wire Line
-	3750 2200 3750 2450
 Wire Wire Line
 	3750 2750 3750 2900
@@
 Text Notes 3050 7550 0    60   ~ 0
 http://www.digikey.com/product-search/en/connectors-interconnects/rectangular-connectors-headers-male-pins/1442547?k=header&k=&pkeyword=header&v=19&FV=1140160%2C1600018%2C1600309%2C160045f%2C8000010%2Cfff40016%2Cfff802f3&mnonly=0&newproducts=0&ColumnSort=0&page=1&quantity=0&ptm=0&fid=0&pageSize=25
+NoConn ~ 3700 2200
+Wire Wire Line
+	3750 2450 3750 2300
+Connection ~ 3750 2300
 $EndSCHEMATC
