File: hardware/PCB/Pyramid/dev10/dev10.kicad_pcb (KiCad board)
At the start: 2 copper layers, 45.9 x 24.5 mm, 13 parts, among them P1 Power, P2 Audio, SW1 WifiRst, U1 LM1117-3.3, U2 ESP-07v2

Commit message: Hårdvara
Parts:
- moved P1 0.82 mm to (201.5, 103.2)
Routing:
- net +5V: track 23.7 -> 21.8 mm
Other:
- outline, holes or cut-outs redrawn
Changed lines of the file:
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@@
     (links 33)
     (no_connects 0)
-    (area 159.132199 90.895099 205.205401 115.556101)
+    (area 159.132199 90.823725 206.751001 115.556101)
     (thickness 1.6)
     (drawings 11)
-    (tracks 156)
+    (tracks 157)
     (zones 0)
     (modules 13)
@@
   )
   (module ASKicadLib:USB_Mini-B_AS (layer F.Cu)
-    (at 201.676 102.4509 180)
+    (at 201.5 103.25 180)
     (descr "USB Mini-B 5-pin SMD connector")
     (tags "USB USB_B USB_Mini connector")
@@
       (net 11 "Net-(R3-Pad2)"))
   )
+  (gr_line (start 205.14 107.11) (end 205.14 115.48) (angle 90) (layer Edge.Cuts) (width 0.15))
+  (gr_line (start 198.87 107.11) (end 205.14 107.11) (angle 90) (layer Edge.Cuts) (width 0.15))
+  (gr_line (start 198.87 99.46) (end 198.87 107.11) (angle 90) (layer Edge.Cuts) (width 0.15))
+  (gr_line (start 205.14 99.46) (end 198.87 99.46) (angle 90) (layer Edge.Cuts) (width 0.15))
+  (gr_line (start 205.14 90.97) (end 205.14 99.46) (angle 90) (layer Edge.Cuts) (width 0.15))
   (gr_text "A/M Sundberg" (at 199.644 114.4016) (layer F.SilkS)
     (effects (font (size 1 1) (thickness 0.25)))
@@
   (gr_line (start 159.2072 115.4811) (end 159.2072 90.9701) (angle 90) (layer Edge.Cuts) (width 0.15))
   (gr_line (start 205.1304 115.4811) (end 159.2072 115.4811) (angle 90) (layer Edge.Cuts) (width 0.15))
-  (gr_line (start 205.1304 106.3752) (end 205.1304 115.4811) (angle 90) (layer Edge.Cuts) (width 0.15))
-  (gr_line (start 199.0979 106.3752) (end 205.1304 106.3752) (angle 90) (layer Edge.Cuts) (width 0.15))
-  (gr_line (start 199.0979 98.6155) (end 199.0979 106.3752) (angle 90) (layer Edge.Cuts) (width 0.15))
-  (gr_line (start 205.1304 98.6155) (end 199.0979 98.6155) (angle 90) (layer Edge.Cuts) (width 0.15))
-  (gr_line (start 205.1304 90.9701) (end 205.1304 98.6155) (angle 90) (layer Edge.Cuts) (width 0.15))
   (gr_line (start 159.258 90.9701) (end 205.1304 90.9701) (angle 90) (layer Edge.Cuts) (width 0.15))
-  (segment (start 190.9064 105.6132) (end 190.9064 108.3564) (width 0.5) (layer F.Cu) (net 1))
-  (segment (start 196.9643 103.8733) (end 198.2216 103.8733) (width 0.5) (layer F.Cu) (net 1))
-  (segment (start 196.3166 104.521) (end 196.9643 103.8733) (width 0.5) (layer F.Cu) (net 1))
-  (segment (start 196.3166 109.4613) (end 196.3166 104.521) (width 0.5) (layer F.Cu) (net 1))
-  (segment (start 195.7578 110.0201) (end 196.3166 109.4613) (width 0.5) (layer F.Cu) (net 1))
-  (segment (start 192.5701 110.0201) (end 195.7578 110.0201) (width 0.5) (layer F.Cu) (net 1))
-  (segment (start 190.9064 108.3564) (end 192.5701 110.0201) (width 0.5) (layer F.Cu) (net 1))
+  (segment (start 190.9064 105.6132) (end 190.9064 108.0264) (width 0.5) (layer F.Cu) (net 1) (status 400000))
+  (segment (start 196.7976 104.6724) (end 198.0456 104.6724) (width 0.5) (layer F.Cu) (net 1) (status 800000))
+  (segment (start 196.11 105.36) (end 196.7976 104.6724) (width 0.5) (layer F.Cu) (net 1))
+  (segment (start 196.11 108.75) (end 196.11 105.36) (width 0.5) (layer F.Cu) (net 1))
+  (segment (start 195.17 109.69) (end 196.11 108.75) (width 0.5) (layer F.Cu) (net 1))
+  (segment (start 192.57 109.69) (end 195.17 109.69) (width 0.5) (layer F.Cu) (net 1))
+  (segment (start 190.9064 108.0264) (end 192.57 109.69) (width 0.5) (layer F.Cu) (net 1))
   (segment (start 187.2107 110.4933) (end 187.2107 109.4613) (width 0.5) (layer F.Cu) (net 1))
   (segment (start 190.9064 107.5944) (end 190.9064 105.6132) (width 0.5) (layer F.Cu) (net 1))
@@
   (segment (start 187.9854 108.6866) (end 189.8142 108.6866) (width 0.5) (layer F.Cu) (net 1))
   (segment (start 187.2107 109.4613) (end 187.9854 108.6866) (width 0.5) (layer F.Cu) (net 1))
+  (segment (start 198.14974 98.79992) (end 198.14974 101.67266) (width 0.5) (layer F.Cu) (net 2) (status C00000))
+  (segment (start 198.14974 101.67266) (end 198.0456 101.7768) (width 0.5) (layer F.Cu) (net 2) (status C00000))
   (segment (start 183.5404 102.0724) (end 186.13124 102.0724) (width 0.5) (layer F.Cu) (net 2))
   (segment (start 190.89624 97.3074) (end 194.0814 97.3074) (width 0.5) (layer B.Cu) (net 2))
@@
   (segment (start 203.4794 98.0059) (end 198.33082 98.0059) (width 0.5) (layer F.Cu) (net 2))
   (segment (start 198.33082 98.0059) (end 198.32574 98.00082) (width 0.5) (layer F.Cu) (net 2))
-  (segment (start 198.2216 100.9777) (end 198.2216 98.10496) (width 0.5) (layer F.Cu) (net 2))
   (segment (start 198.2216 98.10496) (end 198.32574 98.00082) (width 0.5) (layer F.Cu) (net 2))
   (segment (start 197.69074 106.90098) (end 202.78852 106.90098) (width 0.5) (layer F.Cu) (net 2))
