File: hardware/PCB/UsbSticka/01dev/01dev.sch (KiCad schematic (older format))
At the start: 22 parts, among them P1 USB_B, P2 MIC, P3 Debug, SW1 SW_PUSH, SW2 SW_PUSH, U1 LM1117-3.3, U2 MAX9813, U3 ESP-07v2, U4 MCP3201

Commit message: Corr25typ
Parts:
- P1: footprint ASKicadLib:USB_A_AS -> Connect:USB_Micro-B
Changed lines of the file:
@@
 F 0 "P1" H 2900 1600 50  0000 C CNN
 F 1 "USB_B" H 2650 2000 50  0000 C CNN
-F 2 "ASKicadLib:USB_A_AS" V 2650 1700 50  0001 C CNN
+F 2 "Connect:USB_Micro-B" V 2650 1700 50  0001 C CNN
 F 3 "" V 2650 1700 50  0000 C CNN
 	1    2700 1800
@@
 $EndComp
 $Comp
-L GND #PWR5
+L GND #PWR01
 U 1 1 58496CB6
 P 3250 2450
-F 0 "#PWR5" H 3250 2200 50  0001 C CNN
+F 0 "#PWR01" H 3250 2200 50  0001 C CNN
 F 1 "GND" H 3250 2300 50  0000 C CNN
 F 2 "" H 3250 2450 50  0000 C CNN
@@
 $EndComp
 $Comp
-L GND #PWR7
+L GND #PWR02
 U 1 1 58496D02
 P 3850 2350
-F 0 "#PWR7" H 3850 2100 50  0001 C CNN
+F 0 "#PWR02" H 3850 2100 50  0001 C CNN
 F 1 "GND" H 3850 2200 50  0000 C CNN
 F 2 "" H 3850 2350 50  0000 C CNN
@@
 $EndComp
 $Comp
-L GND #PWR8
+L GND #PWR03
 U 1 1 58496D25
 P 4250 2400
-F 0 "#PWR8" H 4250 2150 50  0001 C CNN
+F 0 "#PWR03" H 4250 2150 50  0001 C CNN
 F 1 "GND" H 4250 2250 50  0000 C CNN
 F 2 "" H 4250 2400 50  0000 C CNN
@@
 $EndComp
 $Comp
-L GND #PWR3
+L GND #PWR04
 U 1 1 58496D48
 P 3100 1700
-F 0 "#PWR3" H 3100 1450 50  0001 C CNN
+F 0 "#PWR04" H 3100 1450 50  0001 C CNN
 F 1 "GND" H 3100 1550 50  0000 C CNN
 F 2 "" H 3100 1700 50  0000 C CNN
@@
 NoConn ~ 3000 1800
 $Comp
-L GND #PWR1
+L GND #PWR05
 U 1 1 58496E15
 P 2600 1450
-F 0 "#PWR1" H 2600 1200 50  0001 C CNN
+F 0 "#PWR05" H 2600 1200 50  0001 C CNN
 F 1 "GND" H 2600 1300 50  0000 C CNN
 F 2 "" H 2600 1450 50  0000 C CNN
@@
 $EndComp
 $Comp
-L VCC #PWR11
+L VCC #PWR06
 U 1 1 58496F27
 P 5750 1150
-F 0 "#PWR11" H 5750 1000 50  0001 C CNN
+F 0 "#PWR06" H 5750 1000 50  0001 C CNN
 F 1 "VCC" H 5750 1300 50  0000 C CNN
 F 2 "" H 5750 1150 50  0000 C CNN
@@
 MISO
 $Comp
-L VCC #PWR9
+L VCC #PWR07
 U 1 1 5849724E
 P 4350 1700
-F 0 "#PWR9" H 4350 1550 50  0001 C CNN
+F 0 "#PWR07" H 4350 1550 50  0001 C CNN
 F 1 "VCC" H 4350 1850 50  0000 C CNN
 F 2 "" H 4350 1700 50  0000 C CNN
@@
 $EndComp
 $Comp
-L GND #PWR17
+L GND #PWR08
 U 1 1 58497429
 P 6950 1650
-F 0 "#PWR17" H 6950 1400 50  0001 C CNN
+F 0 "#PWR08" H 6950 1400 50  0001 C CNN
 F 1 "GND" H 6950 1500 50  0000 C CNN
 F 2 "" H 6950 1650 50  0000 C CNN
@@
 $EndComp
 $Comp
-L GND #PWR20
+L GND #PWR09
 U 1 1 58497756
 P 7600 1600
-F 0 "#PWR20" H 7600 1350 50  0001 C CNN
+F 0 "#PWR09" H 7600 1350 50  0001 C CNN
 F 1 "GND" H 7600 1450 50  0000 C CNN
 F 2 "" H 7600 1600 50  0000 C CNN
@@
 $EndComp
 $Comp
-L VCC #PWR23
+L VCC #PWR010
 U 1 1 584977A9
 P 8300 2000
-F 0 "#PWR23" H 8300 1850 50  0001 C CNN
+F 0 "#PWR010" H 8300 1850 50  0001 C CNN
 F 1 "VCC" H 8300 2150 50  0000 C CNN
 F 2 "" H 8300 2000 50  0000 C CNN
@@
 $EndComp
 $Comp
-L GND #PWR19
+L GND #PWR011
 U 1 1 584979DE
 P 7450 2200
-F 0 "#PWR19" H 7450 1950 50  0001 C CNN
+F 0 "#PWR011" H 7450 1950 50  0001 C CNN
 F 1 "GND" H 7450 2050 50  0000 C CNN
 F 2 "" H 7450 2200 50  0000 C CNN
@@
 SS
 $Comp
-L GND #PWR12
+L GND #PWR012
 U 1 1 58497BC9
 P 5750 3050
-F 0 "#PWR12" H 5750 2800 50  0001 C CNN
+F 0 "#PWR012" H 5750 2800 50  0001 C CNN
 F 1 "GND" H 5750 2900 50  0000 C CNN
 F 2 "" H 5750 3050 50  0000 C CNN
@@
 $EndComp
 $Comp
-L GND #PWR14
+L GND #PWR013
 U 1 1 58497DF0
 P 6700 2800
-F 0 "#PWR14" H 6700 2550 50  0001 C CNN
+F 0 "#PWR013" H 6700 2550 50  0001 C CNN
 F 1 "GND" H 6700 2650 50  0000 C CNN
 F 2 "" H 6700 2800 50  0000 C CNN
@@
 SS
 $Comp
-L GND #PWR16
+L GND #PWR014
 U 1 1 58498754
 P 6850 4150
-F 0 "#PWR16" H 6850 3900 50  0001 C CNN
+F 0 "#PWR014" H 6850 3900 50  0001 C CNN
 F 1 "GND" H 6850 4000 50  0000 C CNN
 F 2 "" H 6850 4150 50  0000 C CNN
@@
 $EndComp
 $Comp
-L GND #PWR21
+L GND #PWR015
 U 1 1 58498B1C
 P 7850 4550
-F 0 "#PWR21" H 7850 4300 50  0001 C CNN
+F 0 "#PWR015" H 7850 4300 50  0001 C CNN
 F 1 "GND" H 7850 4400 50  0000 C CNN
 F 2 "" H 7850 4550 50  0000 C CNN
@@
 $EndComp
 $Comp
-L GND #PWR18
+L GND #PWR016
 U 1 1 58498B8F
 P 7300 3500
-F 0 "#PWR18" H 7300 3250 50  0001 C CNN
+F 0 "#PWR016" H 7300 3250 50  0001 C CNN
 F 1 "GND" H 7300 3350 50  0000 C CNN
 F 2 "" H 7300 3500 50  0000 C CNN
@@
 	6700 4700 6750 4700
 $Comp
-L GND #PWR15
+L GND #PWR017
 U 1 1 584993C0
 P 6750 4700
-F 0 "#PWR15" H 6750 4450 50  0001 C CNN
+F 0 "#PWR017" H 6750 4450 50  0001 C CNN
 F 1 "GND" H 6750 4550 50  0000 C CNN
 F 2 "" H 6750 4700 50  0000 C CNN
@@
 Connection ~ 3050 1700
 $Comp
-L GNDA #PWR2
+L GNDA #PWR018
 U 1 1 5849F85B
 P 3050 1650
-F 0 "#PWR2" H 3050 1400 50  0001 C CNN
+F 0 "#PWR018" H 3050 1400 50  0001 C CNN
 F 1 "GNDA" H 3050 1500 50  0000 C CNN
 F 2 "" H 3050 1650 50  0000 C CNN
@@
 	4800 4000 4850 4000
 $Comp
-L GNDA #PWR10
+L GNDA #PWR019
 U 1 1 584C9743
 P 4850 4000
-F 0 "#PWR10" H 4850 3750 50  0001 C CNN
+F 0 "#PWR019" H 4850 3750 50  0001 C CNN
 F 1 "GNDA" H 4850 3850 50  0000 C CNN
 F 2 "" H 4850 4000 50  0000 C CNN
@@
 Connection ~ 3350 4350
 $Comp
-L GNDA #PWR4
+L GNDA #PWR020
 U 1 1 584C9864
 P 3100 4350
-F 0 "#PWR4" H 3100 4100 50  0001 C CNN
+F 0 "#PWR020" H 3100 4100 50  0001 C CNN
 F 1 "GNDA" H 3100 4200 50  0000 C CNN
 F 2 "" H 3100 4350 50  0000 C CNN
@@
 	3450 2000 3450 1900
 $Comp
-L +5V #PWR6
+L +5V #PWR021
 U 1 1 584C9DC3
 P 3450 1900
-F 0 "#PWR6" H 3450 1750 50  0001 C CNN
+F 0 "#PWR021" H 3450 1750 50  0001 C CNN
 F 1 "+5V" H 3450 2040 50  0000 C CNN
 F 2 "" H 3450 1900 50  0000 C CNN
@@
 $EndComp
 $Comp
-L +5V #PWR13
+L +5V #PWR022
 U 1 1 584C9E14
 P 6400 5200
-F 0 "#PWR13" H 6400 5050 50  0001 C CNN
+F 0 "#PWR022" H 6400 5050 50  0001 C CNN
 F 1 "+5V" H 6400 5340 50  0000 C CNN
 F 2 "" H 6400 5200 50  0000 C CNN
@@
 $EndComp
 $Comp
-L +5V #PWR22
+L +5V #PWR023
 U 1 1 584C9E5E
 P 7950 4150
-F 0 "#PWR22" H 7950 4000 50  0001 C CNN
+F 0 "#PWR023" H 7950 4000 50  0001 C CNN
 F 1 "+5V" H 7950 4290 50  0000 C CNN
 F 2 "" H 7950 4150 50  0000 C CNN
