File: hardware/PCB/UsbSticka/01dev/01dev_long_microUSB.kicad_pcb (KiCad board)
At the start: 2 copper layers, 17.7 x 51.8 mm, 23 parts, among them P1 USB_B, P2 MIC, SW1 SW_PUSH, SW2 SW_PUSH, U1 LM1117-3.3, U2 MAX9813, U3 ESP-07v2, U4 MCP3201

Commit message: Corr25typ
Parts:
- removed the P1 at (0.00, 0.00)
- P1: footprint ASKicadLib:USB_A_AS -> Connect:USB_Micro-B
- moved P1 8.08 mm to (150.9, 57.2), turned to 180 degrees
Routing:
- net +5V: track 50.6 -> 55.9 mm
- net GND: vias 3 -> 4

Commit message: Lite Div
Changed lines of the file:
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@@
     (links 49)
     (no_connects 0)
-    (area -7.69987 -9.675001 171.43 106.500001)
+    (area 140.549999 47.75 171.43 106.500001)
     (thickness 1.6)
     (drawings 53)
@@
   (gr_line (start 143.105 100.64) (end 142.23 99.765) (angle 90) (layer F.SilkS) (width 0.127))
   (gr_line (start 159.76 104.6) (end 159.76 104.58) (angle 90) (layer Edge.Cuts) (width 0.15))
-  (gr_text "AHE-Stick\n" (at 151.26 86.53) (layer F.SilkS)
+  (gr_text "AHE-Stick\n" (at 151.3 94.6) (layer F.SilkS)
     (effects (font (size 1 1) (thickness 0.25)))
   )
