File: hardware/PCB/UsbSticka/01dev/02devOPA345.sch (KiCad schematic (older format))
At the start: 22 parts, among them P1 USB_B, P2 MIC, P3 Debug, SW1 SW_PUSH, SW2 SW_PUSH, U1 LM1117-3.3, U2 MAX9813, U3 ESP-07v2, U4 MCP3201

Commit message: StickUppdatering
Parts:
- removed C5: 0,1, Capacitors_SMD:C_0805, symbol C
- removed U2: MAX9813, lab11-ic:SOT-23-8, symbol MAX9813
- added R10: 2k, Resistors_SMD:R_0805, symbol R
- added R6: 820k, Resistors_SMD:R_0805, symbol R
- added R7, R8: 10k, Resistors_SMD:R_0805, symbol R
- added R9: 1k, Resistors_SMD:R_0805, symbol R
- added U2: OPA345, TO_SOT_Packages_SMD:SOT-23-5, symbol OPA345
- C2, C4: value 0,1 -> 4,7
- P1: footprint Connect:USB_Micro-B -> ASKicadLib:USB_A_AS
- R2: value 2,2k -> 10k
Connections:
- net +5V: now also R1.2, R8.1
- net ANALOG: now also R6.1, U2.1 (OUT); no longer C2.2
- net GND: now also C4.1, R10.1, R7.2, U2.2 (V-)
- net MISO: now also R10.2, R9.1; no longer U4.6 (DOut)
- net at C6.2, FB1.1, U4.1 (Vref): now also U2.5 (V+); no longer R2.1
- net at C2.1: now also P2.2 (P2), R1.1
- net at R2.2: now also C2.2
- net at C4.2: now also R7.1, R8.2, U2.3 (+In)
- new net: R9.2, U4.6 (DOut)
- new net: R2.1, R6.2, U2.4 (-In)
- no-connect marks 9 -> 8
Other:
- note added: "3 eller 5 v??\n"
- moved on the sheet: P2
