File: hardware/PCB/UsbSticka/01dev/02devOPA345.sch (KiCad schematic (older format))
At the start: 30 parts, among them P1 USB_B, P2 Debug, P3 MIC, SW1 SW_PUSH, SW2 SW_PUSH, U1 LM1117-3.3, U2 ESP-07v2, U3 OPA345, U4 MCP3201

Commit message: NewPCB Things
Parts:
- gave numbers to parts that had none: 1
Changed lines of the file:
@@
 $EndComp
 $Comp
-L GND #PWR14
+L GND #PWR01
 U 1 1 58496CB6
 P 3250 2450
-F 0 "#PWR14" H 3250 2200 50  0001 C CNN
+F 0 "#PWR01" H 3250 2200 50  0001 C CNN
 F 1 "GND" H 3250 2300 50  0000 C CNN
 F 2 "" H 3250 2450 50  0000 C CNN
@@
 $EndComp
 $Comp
-L GND #PWR11
+L GND #PWR02
 U 1 1 58496D02
 P 3850 2350
-F 0 "#PWR11" H 3850 2100 50  0001 C CNN
+F 0 "#PWR02" H 3850 2100 50  0001 C CNN
 F 1 "GND" H 3850 2200 50  0000 C CNN
 F 2 "" H 3850 2350 50  0000 C CNN
@@
 $EndComp
 $Comp
-L GND #PWR12
+L GND #PWR03
 U 1 1 58496D25
 P 4250 2400
-F 0 "#PWR12" H 4250 2150 50  0001 C CNN
+F 0 "#PWR03" H 4250 2150 50  0001 C CNN
 F 1 "GND" H 4250 2250 50  0000 C CNN
 F 2 "" H 4250 2400 50  0000 C CNN
@@
 $EndComp
 $Comp
-L GND #PWR6
+L GND #PWR04
 U 1 1 58496D48
 P 3100 1700
-F 0 "#PWR6" H 3100 1450 50  0001 C CNN
+F 0 "#PWR04" H 3100 1450 50  0001 C CNN
 F 1 "GND" H 3100 1550 50  0000 C CNN
 F 2 "" H 3100 1700 50  0000 C CNN
@@
 NoConn ~ 3000 1800
 $Comp
-L GND #PWR2
+L GND #PWR05
 U 1 1 58496E15
 P 2600 1450
-F 0 "#PWR2" H 2600 1200 50  0001 C CNN
+F 0 "#PWR05" H 2600 1200 50  0001 C CNN
 F 1 "GND" H 2600 1300 50  0000 C CNN
 F 2 "" H 2600 1450 50  0000 C CNN
@@
 $EndComp
 $Comp
-L VCC #PWR1
+L VCC #PWR06
 U 1 1 58496F27
 P 5750 1150
-F 0 "#PWR1" H 5750 1000 50  0001 C CNN
+F 0 "#PWR06" H 5750 1000 50  0001 C CNN
 F 1 "VCC" H 5750 1300 50  0000 C CNN
 F 2 "" H 5750 1150 50  0000 C CNN
@@
 MISO
 $Comp
-L VCC #PWR7
+L VCC #PWR07
 U 1 1 5849724E
 P 4350 1700
-F 0 "#PWR7" H 4350 1550 50  0001 C CNN
+F 0 "#PWR07" H 4350 1550 50  0001 C CNN
 F 1 "VCC" H 4350 1850 50  0000 C CNN
 F 2 "" H 4350 1700 50  0000 C CNN
@@
 $EndComp
 $Comp
-L GND #PWR5
+L GND #PWR08
 U 1 1 58497429
 P 6950 1650
-F 0 "#PWR5" H 6950 1400 50  0001 C CNN
+F 0 "#PWR08" H 6950 1400 50  0001 C CNN
 F 1 "GND" H 6950 1500 50  0000 C CNN
 F 2 "" H 6950 1650 50  0000 C CNN
@@
 $EndComp
 $Comp
-L GND #PWR3
+L GND #PWR09
 U 1 1 58497756
 P 7600 1600
-F 0 "#PWR3" H 7600 1350 50  0001 C CNN
+F 0 "#PWR09" H 7600 1350 50  0001 C CNN
 F 1 "GND" H 7600 1450 50  0000 C CNN
 F 2 "" H 7600 1600 50  0000 C CNN
@@
 $EndComp
 $Comp
-L VCC #PWR9
+L VCC #PWR010
 U 1 1 584977A9
 P 8300 2000
-F 0 "#PWR9" H 8300 1850 50  0001 C CNN
+F 0 "#PWR010" H 8300 1850 50  0001 C CNN
 F 1 "VCC" H 8300 2150 50  0000 C CNN
 F 2 "" H 8300 2000 50  0000 C CNN
@@
 $EndComp
 $Comp
-L GND #PWR10
+L GND #PWR011
 U 1 1 584979DE
 P 7450 2200
-F 0 "#PWR10" H 7450 1950 50  0001 C CNN
+F 0 "#PWR011" H 7450 1950 50  0001 C CNN
 F 1 "GND" H 7450 2050 50  0000 C CNN
 F 2 "" H 7450 2200 50  0000 C CNN
@@
 SS
 $Comp
-L GND #PWR16
+L GND #PWR012
 U 1 1 58497BC9
 P 5750 3050
-F 0 "#PWR16" H 5750 2800 50  0001 C CNN
+F 0 "#PWR012" H 5750 2800 50  0001 C CNN
 F 1 "GND" H 5750 2900 50  0000 C CNN
 F 2 "" H 5750 3050 50  0000 C CNN
@@
 $EndComp
 $Comp
-L GND #PWR15
+L GND #PWR013
 U 1 1 58497DF0
 P 6700 2800
-F 0 "#PWR15" H 6700 2550 50  0001 C CNN
+F 0 "#PWR013" H 6700 2550 50  0001 C CNN
 F 1 "GND" H 6700 2650 50  0000 C CNN
 F 2 "" H 6700 2800 50  0000 C CNN
@@
 SS
 $Comp
-L GND #PWR23
+L GND #PWR014
 U 1 1 58498754
 P 7950 4800
-F 0 "#PWR23" H 7950 4550 50  0001 C CNN
+F 0 "#PWR014" H 7950 4550 50  0001 C CNN
 F 1 "GND" H 7950 4650 50  0000 C CNN
 F 2 "" H 7950 4800 50  0000 C CNN
@@
 $EndComp
 $Comp
-L GND #PWR19
+L GND #PWR015
 U 1 1 58498B1C
 P 8350 3800
-F 0 "#PWR19" H 8350 3550 50  0001 C CNN
+F 0 "#PWR015" H 8350 3550 50  0001 C CNN
 F 1 "GND" H 8350 3650 50  0000 C CNN
 F 2 "" H 8350 3800 50  0000 C CNN
@@
 $EndComp
 $Comp
-L GND #PWR24
+L GND #PWR016
 U 1 1 584993C0
 P 7450 4850
-F 0 "#PWR24" H 7450 4600 50  0001 C CNN
+F 0 "#PWR016" H 7450 4600 50  0001 C CNN
 F 1 "GND" H 7450 4700 50  0000 C CNN
 F 2 "" H 7450 4850 50  0000 C CNN
@@
 $EndComp
 $Comp
-L GNDA #PWR4
+L GNDA #PWR017
 U 1 1 5849F85B
 P 3050 1650
-F 0 "#PWR4" H 3050 1400 50  0001 C CNN
+F 0 "#PWR017" H 3050 1400 50  0001 C CNN
 F 1 "GNDA" H 3050 1500 50  0000 C CNN
 F 2 "" H 3050 1650 50  0000 C CNN
@@
 $EndComp
 $Comp
-L +5V #PWR8
+L +5V #PWR018
 U 1 1 584C9DC3
 P 3450 1900
-F 0 "#PWR8" H 3450 1750 50  0001 C CNN
+F 0 "#PWR018" H 3450 1750 50  0001 C CNN
 F 1 "+5V" H 3450 2040 50  0000 C CNN
 F 2 "" H 3450 1900 50  0000 C CNN
@@
 $EndComp
 $Comp
-L GNDA #PWR21
+L GNDA #PWR019
 U 1 1 584C9864
 P 2650 4200
-F 0 "#PWR21" H 2650 3950 50  0001 C CNN
+F 0 "#PWR019" H 2650 3950 50  0001 C CNN
 F 1 "GNDA" H 2650 4050 50  0000 C CNN
 F 2 "" H 2650 4200 50  0000 C CNN
@@
 $EndComp
 $Comp
-L GNDA #PWR25
+L GNDA #PWR020
 U 1 1 5883C9E5
 P 3400 5000
-F 0 "#PWR25" H 3400 4750 50  0001 C CNN
+F 0 "#PWR020" H 3400 4750 50  0001 C CNN
 F 1 "GNDA" H 3400 4850 50  0000 C CNN
 F 2 "" H 3400 5000 50  0000 C CNN
@@
 $EndComp
 $Comp
-L VCC #PWR17
+L VCC #PWR021
 U 1 1 5887A831
 P 6300 3500
-F 0 "#PWR17" H 6300 3350 50  0001 C CNN
+F 0 "#PWR021" H 6300 3350 50  0001 C CNN
 F 1 "VCC" H 6300 3650 50  0000 C CNN
 F 2 "" H 6300 3500 50  0000 C CNN
@@
 $EndComp
 $Comp
-L GND #PWR18
+L GND #PWR022
 U 1 1 588A3B8A
 P 4050 3650
-F 0 "#PWR18" H 4050 3400 50  0001 C CNN
+F 0 "#PWR022" H 4050 3400 50  0001 C CNN
 F 1 "GND" H 4050 3500 50  0000 C CNN
 F 2 "" H 4050 3650 50  0000 C CNN
@@
 	6100 4650 6100 4750
 $Comp
-L GND #PWR22
+L GND #PWR023
 U 1 1 588A68A8
 P 6100 4750
-F 0 "#PWR22" H 6100 4500 50  0001 C CNN
+F 0 "#PWR023" H 6100 4500 50  0001 C CNN
 F 1 "GND" H 6100 4600 50  0000 C CNN
 F 2 "" H 6100 4750 50  0000 C CNN
@@
 $EndComp
 $Comp
-L GND #PWR13
+L GND #PWR024
 U 1 1 588A6B83
 P 3050 2450
-F 0 "#PWR13" H 3050 2200 50  0001 C CNN
+F 0 "#PWR024" H 3050 2200 50  0001 C CNN
 F 1 "GND" H 3050 2300 50  0000 C CNN
 F 2 "" H 3050 2450 50  0000 C CNN
@@
 Connection ~ 6300 3550
 $Comp
-L C C?
+L C C6
 U 1 1 588CCCA0
 P 6050 3550
-F 0 "C?" H 6075 3650 50  0000 L CNN
+F 0 "C6" H 6075 3650 50  0000 L CNN
 F 1 "0,1uF" H 6075 3450 50  0000 L CNN
 F 2 "Capacitors_SMD:C_0805" H 6088 3400 50  0001 C CNN
@@
 	5900 3550 5850 3550
 $Comp
-L GND #PWR?
+L GND #PWR025
 U 1 1 588CCE7C
 P 5850 3550
-F 0 "#PWR?" H 5850 3300 50  0001 C CNN
+F 0 "#PWR025" H 5850 3300 50  0001 C CNN
 F 1 "GND" H 5850 3400 50  0000 C CNN
 F 2 "" H 5850 3550 50  0000 C CNN
