File: hardware/PCB/UsbSticka/01dev/02dev.sch (KiCad schematic (older format))
At the start: 22 parts, among them P1 USB_B, P2 MIC, P3 Debug, SW1 SW_PUSH, SW2 SW_PUSH, U1 LM1117-3.3, U2 MAX9813, U3 ESP-07v2, U4 MCP3201

Commit message: StickUppdatering
Parts:
- P1: footprint Connect:USB_Micro-B -> ASKicadLib:USB_A_AS
Changed lines of the file:
@@
 LIBS:contrib
 LIBS:valves
-LIBS:andreas_footprints
-LIBS:ferrite
-LIBS:01dev-cache
+LIBS:02dev-cache
 EELAYER 25 0
 EELAYER END
@@
 F 0 "P1" H 2900 1600 50  0000 C CNN
 F 1 "USB_B" H 2650 2000 50  0000 C CNN
-F 2 "Connect:USB_Micro-B" V 2650 1700 50  0001 C CNN
+F 2 "ASKicadLib:USB_A_AS" V 2650 1700 50  0001 C CNN
 F 3 "" V 2650 1700 50  0000 C CNN
 	1    2700 1800

Commit message: New hardware
Parts:
- added C8: 0,1, Capacitors_SMD:C_0805, symbol C
- added C9: 10uF, Capacitors_SMD:C_0805, symbol C
- added R6, R7, R8: 1k, Resistors_SMD:R_0805, symbol R
Connections:
- net ANALOG: now also C2.1, U2.1 (OUT); no longer C2.2, U4.2 (Vin+)
- net GND: now also C8.1, C9.2, R8.2
- net MISO: now also R6.1, R7.1; no longer U4.6 (DOut)
- net at C5.2, C6.2, FB1.1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: now also C9.1
- net at C4.2, U2.6 (IN1): now also C8.2
- new net: C2.2, U4.2 (Vin+)
- new net: R6.2, U4.6 (DOut)
- new net: R7.2, R8.1
Other:
- moved on the sheet: C2
Changed lines of the file:
@@
 Text GLabel 7300 4600 3    60   Input ~ 0
 SCLK
-Text GLabel 7400 4600 3    60   Input ~ 0
+Text GLabel 7400 5550 3    60   Input ~ 0
 MISO
 Text GLabel 7500 4600 3    60   Input ~ 0
@@
 	7300 4550 7300 4600
 Wire Wire Line
-	7400 4550 7400 4600
+	7400 4550 7400 4900
 Wire Wire Line
 	7500 4550 7500 4600
@@
 	7300 3550 7300 3500
 Wire Wire Line
-	7500 3550 7500 3500
-Text GLabel 7500 3500 1    60   Input ~ 0
+	7500 3200 7500 3550
+Text GLabel 6150 3450 0    60   Input ~ 0
 ANALOG
 $Comp
@@
 $EndComp
 Wire Wire Line
-	4100 4200 4050 4200
-Wire Wire Line
-	4050 4200 4050 4150
+	4050 4200 4100 4200
+Wire Wire Line
+	4050 3800 4050 4200
 $Comp
 L C C2
 U 1 1 584C93B0
-P 4050 4000
-F 0 "C2" H 4075 4100 50  0000 L CNN
-F 1 "0,1" H 4075 3900 50  0000 L CNN
-F 2 "Capacitors_SMD:C_0805" H 4088 3850 50  0001 C CNN
-F 3 "" H 4050 4000 50  0000 C CNN
-	1    4050 4000
-	-1   0    0    1
-$EndComp
-Wire Wire Line
-	4050 3850 4050 3800
+P 6450 3450
+F 0 "C2" H 6475 3550 50  0000 L CNN
+F 1 "0,1" H 6475 3350 50  0000 L CNN
+F 2 "Capacitors_SMD:C_0805" H 6488 3300 50  0001 C CNN
+F 3 "" H 6450 3450 50  0000 C CNN
+	1    6450 3450
+	0    -1   -1   0
+$EndComp
 Wire Wire Line
 	4050 3800 4100 3800
@@
 $EndComp
 Wire Wire Line
-	4100 4350 3100 4350
+	3100 4350 4100 4350
 Wire Wire Line
 	3350 3700 3350 4350
@@
 	3650 3600 3650 3500
 Wire Wire Line
-	5450 3500 5450 4450
-Wire Wire Line
 	5450 4450 5200 4450
 $Comp
@@
 	0    1    1    0
 $EndComp
+$Comp
+L R R6
+U 1 1 5887B50C
+P 7400 5050
+F 0 "R6" V 7480 5050 50  0000 C CNN
+F 1 "1k" V 7400 5050 50  0000 C CNN
+F 2 "Resistors_SMD:R_0805" V 7330 5050 50  0001 C CNN
+F 3 "" H 7400 5050 50  0000 C CNN
+	1    7400 5050
+	-1   0    0    1
+$EndComp
+$Comp
+L R R7
+U 1 1 5887B6CD
+P 7600 5250
+F 0 "R7" V 7680 5250 50  0000 C CNN
+F 1 "1k" V 7600 5250 50  0000 C CNN
+F 2 "Resistors_SMD:R_0805" V 7530 5250 50  0001 C CNN
+F 3 "" H 7600 5250 50  0000 C CNN
+	1    7600 5250
+	0    -1   -1   0
+$EndComp
+$Comp
+L R R8
+U 1 1 5887B859
+P 7950 5250
+F 0 "R8" V 8030 5250 50  0000 C CNN
+F 1 "1k" V 7950 5250 50  0000 C CNN
+F 2 "Resistors_SMD:R_0805" V 7880 5250 50  0001 C CNN
+F 3 "" H 7950 5250 50  0000 C CNN
+	1    7950 5250
+	0    -1   -1   0
+$EndComp
+$Comp
+L GND #PWR024
+U 1 1 5887B8D0
+P 8150 5250
+F 0 "#PWR024" H 8150 5000 50  0001 C CNN
+F 1 "GND" H 8150 5100 50  0000 C CNN
+F 2 "" H 8150 5250 50  0000 C CNN
+F 3 "" H 8150 5250 50  0000 C CNN
+	1    8150 5250
+	0    -1   -1   0
+$EndComp
+Wire Wire Line
+	8150 5250 8100 5250
+Wire Wire Line
+	7800 5250 7750 5250
+Wire Wire Line
+	7400 5200 7400 5550
+Wire Wire Line
+	7450 5250 7400 5250
+Connection ~ 7400 5250
+Wire Wire Line
+	7500 3200 7100 3200
+Wire Wire Line
+	7100 3200 7100 3450
+Wire Wire Line
+	7100 3450 6600 3450
+Wire Wire Line
+	5450 3500 5450 4450
+Wire Wire Line
+	6150 3450 6300 3450
+Wire Wire Line
+	5400 4450 5400 4850
+Connection ~ 5400 4450
+$Comp
+L C C8
+U 1 1 5889159D
+P 5400 5000
+F 0 "C8" H 5425 5100 50  0000 L CNN
+F 1 "0,1" H 5425 4900 50  0000 L CNN
+F 2 "Capacitors_SMD:C_0805" H 5438 4850 50  0001 C CNN
+F 3 "" H 5400 5000 50  0000 C CNN
+	1    5400 5000
+	-1   0    0    1
+$EndComp
+$Comp
+L GND #PWR025
+U 1 1 58891619
+P 5400 5150
+F 0 "#PWR025" H 5400 4900 50  0001 C CNN
+F 1 "GND" H 5400 5000 50  0000 C CNN
+F 2 "" H 5400 5150 50  0000 C CNN
+F 3 "" H 5400 5150 50  0000 C CNN
+	1    5400 5150
+	1    0    0    -1
+$EndComp
+$Comp
+L C C9
+U 1 1 58891A5F
+P 6050 4000
+F 0 "C9" H 6075 4100 50  0000 L CNN
+F 1 "10uF" H 6075 3900 50  0000 L CNN
+F 2 "Capacitors_SMD:C_0805" H 6088 3850 50  0001 C CNN
+F 3 "" H 6050 4000 50  0000 C CNN
+	1    6050 4000
+	-1   0    0    1
+$EndComp
+$Comp
+L GND #PWR026
+U 1 1 58891AF6
+P 6050 3800
+F 0 "#PWR026" H 6050 3550 50  0001 C CNN
+F 1 "GND" H 6050 3650 50  0000 C CNN
+F 2 "" H 6050 3800 50  0000 C CNN
+F 3 "" H 6050 3800 50  0000 C CNN
+	1    6050 3800
+	-1   0    0    1
+$EndComp
+Wire Wire Line
+	6050 3800 6050 3850
+Wire Wire Line
+	6050 4150 6050 4200
+Connection ~ 6050 4200
 $EndSCHEMATC
