File: hardware/PCB/UsbSticka/01dev/02devOPAdual.sch (KiCad schematic (older format))
At the start: 30 parts, among them P1 USB_B, P2 Debug, P3 MIC, SW1 SW_PUSH, SW2 SW_PUSH, U1 LM1117-3.3, U2 ESP-07v2, U3 OPA345, U4 MCP3201

Commit message: New hardware
Parts:
- removed C8: 3300pF, Capacitors_SMD:C_0805, symbol C
- added R10: 51k, Resistors_SMD:R_0805, symbol R
- added R11: 510k, Resistors_SMD:R_0805, symbol R
- added R12: 150k, Resistors_SMD:R_0805, symbol R
- added U5: OPA345, TO_SOT_Packages_SMD:SOT-23-5, symbol OPA345
- C3: value 0,1 -> C
- C4: value 0,1 -> 1000pF
- C7: value 4,7 -> 33pF
- R4: value 820k -> 20k
- R5: value 2,2k -> 1,5k
- R6, R9: value 10k -> 1M
- R7: value 10k -> 20k
- R8: value 500 -> 100k
- gave numbers to parts that had none: 1
- renumbered SW1 to WifiSw1
Connections:
- net GND: now also C4.1, R4.1, U5.2 (V-); no longer C4.2, U3.2 (V-)
- net at C10.2, C5.2, FB1.1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: now also R7.2; no longer C4.1
- net at U4.2 (Vin+): now also C7.2, R11.2, U5.1 (OUT); no longer R8.1
- net at P3.2 (P2), R5.1: now also C3.2; no longer C7.1
- net at R8.2, U3.1 (OUT): now also R10.1; no longer C3.1, R4.1
- net at R4.2, R7.1, U3.4 (IN-): now also R8.1; no longer C3.2
- net at C9.2, R6.2, R9.1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: now also C3.1, U5.3 (IN+)
- new net: C4.2, R10.2, R11.1, R12.1
- new net: C7.1, R12.2, U5.4 (IN-)
Other:
- moved on the sheet: C6, C9, FB1, P3, R5, R6, R7, R9, U3

Commit message: NewPCB Things
Parts:
- C3: value C -> 1000pF
Changed lines of the file:
@@
 P 1550 4450
 F 0 "C3" H 1575 4550 50  0000 L CNN
-F 1 "C" H 1575 4350 50  0000 L CNN
+F 1 "1000pF" H 1575 4350 50  0000 L CNN
 F 2 "Capacitors_SMD:C_0805" H 1588 4300 50  0001 C CNN
 F 3 "" H 1550 4450 50  0000 C CNN

Commit message: Dev08
Parts:
- C1, C10, C11, C2, C3, C4, C5, C6, C7, C9: footprint Capacitors_SMD:C_0805 -> Capacitors_SMD:C_0805_HandSoldering
- Flash1: renamed from SW2; footprint Buttons_Switches_SMD:SW_SPST_EVQPE1 -> Pin_Headers:Pin_Header_Straight_1x02_Pitch2.54mm
- R1, R10, R11, R12, R2, R3, R4, R5, R6, R7, R8, R9: footprint Resistors_SMD:R_0805 -> Resistors_SMD:R_0805_HandSoldering
- U3: footprint TO_SOT_Packages_SMD:SOT-23-5 -> TO_SOT_Packages_SMD:SOT-23-5_HandSoldering
- Wifi1: renamed from WifiSw1; footprint Buttons_Switches_SMD:SW_SPST_EVQPE1 -> ASKicadLib:SW_PUSH_AS
Changed lines of the file:
@@
 F 0 "C2" H 3275 2350 50  0000 L CNN
 F 1 "10uF" H 3275 2150 50  0000 L CNN
-F 2 "Capacitors_SMD:C_0805" H 3288 2100 50  0001 C CNN
+F 2 "Capacitors_SMD:C_0805_HandSoldering" H 3288 2100 50  0001 C CNN
 F 3 "" H 3250 2250 50  0000 C CNN
 	1    3250 2250
@@
 F 0 "C1" H 4275 2300 50  0000 L CNN
 F 1 "0,1uF" H 4275 2100 50  0000 L CNN
-F 2 "Capacitors_SMD:C_0805" H 4288 2050 50  0001 C CNN
+F 2 "Capacitors_SMD:C_0805_HandSoldering" H 4288 2050 50  0001 C CNN
 F 3 "" H 4250 2200 50  0000 C CNN
 	1    4250 2200
@@
 F 0 "R2" V 4680 2000 50  0000 C CNN
 F 1 "10k" V 4600 2000 50  0000 C CNN
-F 2 "Resistors_SMD:R_0805" V 4530 2000 50  0001 C CNN
+F 2 "Resistors_SMD:R_0805_HandSoldering" V 4530 2000 50  0001 C CNN
 F 3 "" H 4600 2000 50  0000 C CNN
 	1    4600 2000
@@
 F 0 "R1" V 7680 1800 50  0000 C CNN
 F 1 "10k" V 7600 1800 50  0000 C CNN
-F 2 "Resistors_SMD:R_0805" V 7530 1800 50  0001 C CNN
+F 2 "Resistors_SMD:R_0805_HandSoldering" V 7530 1800 50  0001 C CNN
 F 3 "" H 7600 1800 50  0000 C CNN
 	1    7600 1800
@@
 $EndComp
 $Comp
-L SW_PUSH WifiSw1
+L SW_PUSH Wifi1
 U 1 1 5849753C
 P 7950 2000
-F 0 "WifiSw1" H 8100 2110 50  0000 C CNN
+F 0 "Wifi1" H 8100 2110 50  0000 C CNN
 F 1 "SW_PUSH" H 7950 1920 50  0000 C CNN
-F 2 "Buttons_Switches_SMD:SW_SPST_EVQPE1" H 7950 2000 50  0001 C CNN
+F 2 "ASKicadLib:SW_PUSH_AS" H 7950 2000 50  0001 C CNN
 F 3 "" H 7950 2000 50  0000 C CNN
 	1    7950 2000
@@
 NoConn ~ 6650 2300
 $Comp
-L SW_PUSH SW2
+L SW_PUSH Flash1
 U 1 1 5849792E
 P 7100 2200
-F 0 "SW2" H 7250 2310 50  0000 C CNN
+F 0 "Flash1" H 7250 2310 50  0000 C CNN
 F 1 "SW_PUSH" H 7100 2120 50  0000 C CNN
-F 2 "Buttons_Switches_SMD:SW_SPST_EVQPE1" H 7100 2200 50  0001 C CNN
+F 2 "Pin_Headers:Pin_Header_Straight_1x02_Pitch2.54mm" H 7100 2200 50  0001 C CNN
 F 3 "" H 7100 2200 50  0000 C CNN
 	1    7100 2200
@@
 F 0 "R3" V 6780 2600 50  0000 C CNN
 F 1 "10k" V 6700 2600 50  0000 C CNN
-F 2 "Resistors_SMD:R_0805" V 6630 2600 50  0001 C CNN
+F 2 "Resistors_SMD:R_0805_HandSoldering" V 6630 2600 50  0001 C CNN
 F 3 "" H 6700 2600 50  0000 C CNN
 	1    6700 2600
@@
 F 0 "C5" H 8175 3900 50  0000 L CNN
 F 1 "0,1" H 8175 3700 50  0000 L CNN
-F 2 "Capacitors_SMD:C_0805" H 8188 3650 50  0001 C CNN
+F 2 "Capacitors_SMD:C_0805_HandSoldering" H 8188 3650 50  0001 C CNN
 F 3 "" H 8150 3800 50  0000 C CNN
 	1    8150 3800
@@
 F 0 "C10" H 7625 4950 50  0000 L CNN
 F 1 "0,1" H 7625 4750 50  0000 L CNN
-F 2 "Capacitors_SMD:C_0805" H 7638 4700 50  0001 C CNN
+F 2 "Capacitors_SMD:C_0805_HandSoldering" H 7638 4700 50  0001 C CNN
 F 3 "" H 7600 4850 50  0000 C CNN
 	1    7600 4850
@@
 F 0 "R7" V 2430 4100 50  0000 C CNN
 F 1 "20k" V 2350 4100 50  0000 C CNN
-F 2 "Resistors_SMD:R_0805" V 2280 4100 50  0001 C CNN
+F 2 "Resistors_SMD:R_0805_HandSoldering" V 2280 4100 50  0001 C CNN
 F 3 "" H 2350 4100 50  0000 C CNN
 	1    2350 4100
@@
 F 0 "R9" V 1980 4750 50  0000 C CNN
 F 1 "1M" V 1900 4750 50  0000 C CNN
-F 2 "Resistors_SMD:R_0805" V 1830 4750 50  0001 C CNN
+F 2 "Resistors_SMD:R_0805_HandSoldering" V 1830 4750 50  0001 C CNN
 F 3 "" H 1900 4750 50  0000 C CNN
 	1    1900 4750
@@
 F 0 "R6" V 1980 4100 50  0000 C CNN
 F 1 "1M" V 1900 4100 50  0000 C CNN
-F 2 "Resistors_SMD:R_0805" V 1830 4100 50  0001 C CNN
+F 2 "Resistors_SMD:R_0805_HandSoldering" V 1830 4100 50  0001 C CNN
 F 3 "" H 1900 4100 50  0000 C CNN
 	1    1900 4100
@@
 F 0 "C9" H 1725 4850 50  0000 L CNN
 F 1 "4,7" H 1725 4650 50  0000 L CNN
-F 2 "Capacitors_SMD:C_0805" H 1738 4600 50  0001 C CNN
+F 2 "Capacitors_SMD:C_0805_HandSoldering" H 1738 4600 50  0001 C CNN
 F 3 "" H 1700 4750 50  0000 C CNN
 	1    1700 4750
@@
 F 0 "C11" H 3075 2350 50  0000 L CNN
 F 1 "0,1uF" H 3075 2150 50  0000 L CNN
-F 2 "Capacitors_SMD:C_0805" H 3088 2100 50  0001 C CNN
+F 2 "Capacitors_SMD:C_0805_HandSoldering" H 3088 2100 50  0001 C CNN
 F 3 "" H 3050 2250 50  0000 C CNN
 	1    3050 2250
@@
 F 0 "C6" H 6475 3650 50  0000 L CNN
 F 1 "0,1uF" H 6475 3450 50  0000 L CNN
-F 2 "Capacitors_SMD:C_0805" H 6488 3400 50  0001 C CNN
+F 2 "Capacitors_SMD:C_0805_HandSoldering" H 6488 3400 50  0001 C CNN
 F 3 "" H 6450 3550 50  0000 C CNN
 	1    6450 3550
@@
 F 0 "U3" H 3400 4250 50  0000 C CNN
 F 1 "OPA345" V 3150 4250 50  0000 C CNN
-F 2 "TO_SOT_Packages_SMD:SOT-23-5" H 3600 4000 50  0001 C CIN
+F 2 "TO_SOT_Packages_SMD:SOT-23-5_HandSoldering" H 3600 4000 50  0001 C CIN
 F 3 "" H 3250 4250 50  0000 C CNN
 	1    3250 4250
@@
 F 0 "R5" V 1330 4100 50  0000 C CNN
 F 1 "1,5k" V 1250 4100 50  0000 C CNN
-F 2 "Resistors_SMD:R_0805" V 1180 4100 50  0001 C CNN
+F 2 "Resistors_SMD:R_0805_HandSoldering" V 1180 4100 50  0001 C CNN
 F 3 "" H 1250 4100 50  0000 C CNN
 	1    1250 4100
@@
 F 0 "C3" H 1575 4550 50  0000 L CNN
 F 1 "1000pF" H 1575 4350 50  0000 L CNN
-F 2 "Capacitors_SMD:C_0805" H 1588 4300 50  0001 C CNN
+F 2 "Capacitors_SMD:C_0805_HandSoldering" H 1588 4300 50  0001 C CNN
 F 3 "" H 1550 4450 50  0000 C CNN
 	1    1550 4450
@@
 F 0 "R4" V 2430 4900 50  0000 C CNN
 F 1 "20k" V 2350 4900 50  0000 C CNN
-F 2 "Resistors_SMD:R_0805" V 2280 4900 50  0001 C CNN
+F 2 "Resistors_SMD:R_0805_HandSoldering" V 2280 4900 50  0001 C CNN
 F 3 "" H 2350 4900 50  0000 C CNN
 	1    2350 4900
@@
 F 0 "R8" V 3030 4800 50  0000 C CNN
 F 1 "100k" V 2950 4800 50  0000 C CNN
-F 2 "Resistors_SMD:R_0805" V 2880 4800 50  0001 C CNN
+F 2 "Resistors_SMD:R_0805_HandSoldering" V 2880 4800 50  0001 C CNN
 F 3 "" H 2950 4800 50  0000 C CNN
 	1    2950 4800
@@
 F 0 "R10" V 4180 4250 50  0000 C CNN
 F 1 "51k" V 4100 4250 50  0000 C CNN
-F 2 "Resistors_SMD:R_0805" V 4030 4250 50  0001 C CNN
+F 2 "Resistors_SMD:R_0805_HandSoldering" V 4030 4250 50  0001 C CNN
 F 3 "" H 4100 4250 50  0000 C CNN
 	1    4100 4250
@@
 F 0 "R12" V 4580 4250 50  0000 C CNN
 F 1 "150k" V 4500 4250 50  0000 C CNN
-F 2 "Resistors_SMD:R_0805" V 4430 4250 50  0001 C CNN
+F 2 "Resistors_SMD:R_0805_HandSoldering" V 4430 4250 50  0001 C CNN
 F 3 "" H 4500 4250 50  0000 C CNN
 	1    4500 4250
@@
 F 0 "C4" H 4325 4600 50  0000 L CNN
 F 1 "1000pF" H 4325 4400 50  0000 L CNN
-F 2 "Capacitors_SMD:C_0805" H 4338 4350 50  0001 C CNN
+F 2 "Capacitors_SMD:C_0805_HandSoldering" H 4338 4350 50  0001 C CNN
 F 3 "" H 4300 4500 50  0000 C CNN
 	1    4300 4500
@@
 F 0 "R11" V 4580 3750 50  0000 C CNN
 F 1 "510k" V 4500 3750 50  0000 C CNN
-F 2 "Resistors_SMD:R_0805" V 4430 3750 50  0001 C CNN
+F 2 "Resistors_SMD:R_0805_HandSoldering" V 4430 3750 50  0001 C CNN
 F 3 "" H 4500 3750 50  0000 C CNN
 	1    4500 3750
@@
 F 0 "C7" H 5575 4050 50  0000 L CNN
 F 1 "33pF" H 5575 3850 50  0000 L CNN
-F 2 "Capacitors_SMD:C_0805" H 5588 3800 50  0001 C CNN
+F 2 "Capacitors_SMD:C_0805_HandSoldering" H 5588 3800 50  0001 C CNN
 F 3 "" H 5550 3950 50  0000 C CNN
 	1    5550 3950
