File: hardware/PCB/UsbSticka/02dev/02dev.kicad_pcb (KiCad board)
At the start: 2 copper layers, 17.7 x 51.8 mm, 22 parts, among them P1 USB_B, P2 MIC, SW1 SW_PUSH, SW2 SW_PUSH, U1 LM1117-3.3, U2 MAX9813, U3 ESP-07v2, U4 MCP3201

Commit message: Lite Div
Parts:
- P1: footprint Connect:USB_Micro-B -> ASKicadLib:USB_A_AS
- moved P1 8.08 mm to (150.8, 49.1), turned to 0 degrees
- moved C8 5.15 mm to (148.7, 89.5)
- moved FB1 4.69 mm to (144.4, 90.2), turned to 90 degrees
- moved U2 2.46 mm to (149.8, 99.7)
- moved C3 2.16 mm to (151.8, 90.5), turned to 180 degrees
- moved R2 2.05 mm to (146.0, 98.1)
- moved U4 2.05 mm to (149.7, 98.6)
- moved C9 0.88 mm to (143.3, 101.8)
- moved R5 0.79 mm to (154.8, 89.6)
- moved R1 0.70 mm to (151.8, 88.3), turned to 0 degrees
- moved C2 0.38 mm to (157.3, 102.5)
- moved C5 0.18 mm to (157.3, 100.0)
Routing:
- net Net-(C3-Pad2): track 17.0 -> 13.6 mm
- net Net-(C5-Pad2): track 33.0 -> 36.0 mm
- net +5V: track 55.9 -> 53.3 mm
- net VCC: track 53.8 -> 52.3 mm
- net Net-(C3-Pad1): track 10.7 -> 9.25 mm
- net ANALOG: track 13.5 -> 12.1 mm
- net Net-(R1-Pad1): track 17.6 -> 16.4 mm, vias 2 -> 0
- net Net-(R2-Pad2): track 2.83 -> 4.03 mm
- net Net-(SW1-Pad1): track 30.7 -> 31.8 mm
- net GND: track 142.1 -> 141.0 mm, vias 4 -> 3
- net Net-(C2-Pad1): track 8.60 -> 7.73 mm
- net MISO: track 15.2 -> 14.4 mm, vias 2 -> 1
Other:
- board size 17.7 x 51.8 mm -> 17.7 x 49.9 mm
- board text added: "By Sundberg AHE-Stick"
- board text removed: "AHE-Stick"
