File: hardware/PCB/UsbSticka/02dev/02dev_long.kicad_pcb (KiCad board)
At the start: 2 copper layers, 17.7 x 51.8 mm, 22 parts, among them P1 USB_B, P2 MIC, SW1 SW_PUSH, SW2 SW_PUSH, U1 LM1117-3.3, U2 MAX9813, U3 ESP-07v2, U4 MCP3201

Commit message: Lite Div
Parts:
- removed Debug: Debug, Socket_Strips:Socket_Strip_Straight_1x03
- added C6: 100pF, Capacitors_SMD:C_0805, B.Cu at (157.0, 101.5)
- added P3: Debug, Socket_Strips:Socket_Strip_Straight_1x03, F.Cu at (153.6, 76.9)
- added R3: 10k, Resistors_SMD:R_0805, B.Cu at (153.2, 101.6)
- added R7: 100k, Resistors_SMD:R_0805, B.Cu at (157.0, 99.5)
- added R8: 1M, Resistors_SMD:R_0805, B.Cu at (169.5, 90.7)
- added R9: 1M, Resistors_SMD:R_0805, B.Cu at (168.2, 88.1)
- C3: value 0,1 -> 1uF
- C5: value 0,1 -> 0,01; moved to B.Cu
- R1, R2: value 2,2k -> 2k
- U2: value MAX9813 -> MAX4466; footprint lab11-ic:SOT-23-8 -> TO_SOT_Packages_SMD:SC-70-5
- moved FB1 30.6 mm to (176.1, 103.5)
- moved R1 25.9 mm to (178.0, 92.1)
- moved R2 19.8 mm to (163.8, 108.8)
- moved C8 19.1 mm to (170.6, 98.4)
- moved C5 17.5 mm to (170.3, 88.2), turned to 270 degrees
- moved C2 12.1 mm to (169.4, 102.2)
- moved C3 10.6 mm to (153.2, 99.5), turned to 0 degrees
- moved U2 8.89 mm to (157.1, 103.7)
- moved P1 0.16 mm to (151.0, 57.2)
Connections:
- C2 pad 2: ANALOG -> GND
- C5 pad 1: GND -> Net-(C5-Pad1)
- C8 pad 2: Net-(C5-Pad2) -> Net-(C8-Pad2)
- C9 pad 2: +5V -> VCC
- FB1 pad 1: Net-(C5-Pad2) -> Net-(C8-Pad2)
- FB1 pad 2: +5V -> VCC
- P2 pad 2: Net-(C3-Pad1) -> Net-(C5-Pad2)
- R1 pad 1: Net-(R1-Pad1) -> VCC
- R1 pad 2: Net-(C3-Pad1) -> Net-(C2-Pad1)
- R2 pad 1: Net-(C5-Pad2) -> Net-(C2-Pad1)
- R2 pad 2: Net-(R2-Pad2) -> Net-(C5-Pad2)
- U2 pad 1: Net-(C2-Pad1) -> Net-(C5-Pad1)
- U2 pad 3: Net-(C5-Pad2) -> Net-(C3-Pad2)
- U2 pad 4: Net-(R2-Pad2) -> ANALOG
- U2 pad 5: (no net) -> Net-(C8-Pad2)
- U4 pad 1: Net-(C5-Pad2) -> Net-(C8-Pad2)
- U4 pad 8: +5V -> VCC
Routing:
- net +5V: track 55.9 -> 6.36 mm, vias 1 -> 0
- net Net-(C5-Pad2): track 33.0 -> 0.00 mm, vias 1 -> 0
- net Net-(R1-Pad1): track 17.6 -> 0.00 mm, vias 2 -> 0
- net Net-(C3-Pad2): track 17.0 -> 5.34 mm
- net VCC: track 53.8 -> 65.2 mm
- net Net-(C3-Pad1): track 10.7 -> 2.12 mm
- net Net-(C2-Pad1): track 8.60 -> 0.00 mm, vias 1 -> 0
- net ANALOG: track 13.5 -> 18.3 mm, vias 1 -> 0
- net Net-(C5-Pad1): track 0.00 -> 3.60 mm
- net GND: track 142.1 -> 139.2 mm, vias 4 -> 2
- net Net-(R2-Pad2): track 2.83 -> 0.00 mm
- net MISO: track 15.2 -> 16.0 mm, vias 2 -> 1

Commit message: Firmware07 and Pics
Parts:
- C2: moved to B.Cu
- moved R1 24.1 mm to (153.9, 91.6), turned to 0 degrees
- moved R2 23.3 mm to (154.0, 87.7), turned to 180 degrees
- moved C8 21.9 mm to (149.7, 91.8), turned to 0 degrees
- moved C2 19.9 mm to (153.9, 89.6), turned to 180 degrees
- moved R8 19.7 mm to (149.8, 89.8), turned to 0 degrees
- moved R9 18.4 mm to (149.8, 87.8), turned to 180 degrees
- moved U2 12.4 mm to (145.8, 98.7), turned to 0 degrees
- moved R3 4.54 mm to (149.1, 99.7)
- moved R7 4.54 mm to (152.8, 97.6)
- moved C3 4.54 mm to (149.1, 97.6)
- moved C6 4.54 mm to (152.9, 99.5)
- moved R5 2.62 mm to (154.2, 93.0), turned to 180 degrees
- moved U4 2.35 mm to (150.9, 98.7)
- moved C9 0.15 mm to (143.5, 102.9)
Routing:
- net GND: track 139.2 -> 108.5 mm, vias 2 -> 1
- net SS: track 16.5 -> 0.28 mm, vias 1 -> 0
- net MISO: track 16.0 -> 0.74 mm, vias 1 -> 0
- net SCLK: track 15.0 -> 0.00 mm
- net VCC: track 65.2 -> 76.8 mm
- net ANALOG: track 18.3 -> 13.7 mm, vias 0 -> 1
- net Net-(C8-Pad2): track 0.39 -> 4.22 mm
- net Net-(C3-Pad2): track 5.34 -> 8.64 mm
- net Net-(C5-Pad1): track 3.60 -> 2.05 mm
