File: hardware/PCB/UsbSticka/03dev/03devOPA345.sch (KiCad schematic (older format))
At the start: 33 parts, among them P1 USB_B, P2 Debug, P3 MIC, SW2 SW_PUSH, U1 LM1117-3.3, U2 ESP-07v2, U3 OPA345, U4 MCP3201, U5 OPA345

Commit message: Dev08
Parts:
- removed C6: 0,1uF, Capacitors_SMD:C_0805, symbol C
- removed R10: 51k, Resistors_SMD:R_0805, symbol R
- removed R11: 510k, Resistors_SMD:R_0805, symbol R
- removed R12: 150k, Resistors_SMD:R_0805, symbol R
- removed U5: OPA345, TO_SOT_Packages_SMD:SOT-23-5, symbol OPA345
- added C8: 3300pF, Capacitors_SMD:C_0805_HandSoldering, symbol C
- C1, C10, C11, C2, C5, C9: footprint Capacitors_SMD:C_0805 -> Capacitors_SMD:C_0805_HandSoldering
- C3, C4: value 1000pF -> 0,1; footprint Capacitors_SMD:C_0805 -> Capacitors_SMD:C_0805_HandSoldering
- C7: value 33pF -> 4,7; footprint Capacitors_SMD:C_0805 -> Capacitors_SMD:C_0805_HandSoldering
- R1, R2, R3: footprint Resistors_SMD:R_0805 -> Resistors_SMD:R_0805_HandSoldering
- R4: value 20k -> 820k; footprint Resistors_SMD:R_0805 -> Resistors_SMD:R_0805_HandSoldering
- R5: value 1,5k -> 2,2k; footprint Resistors_SMD:R_0805 -> Resistors_SMD:R_0805_HandSoldering
- R6, R9: value 1M -> 10k; footprint Resistors_SMD:R_0805 -> Resistors_SMD:R_0805_HandSoldering
- R7: value 20k -> 10k; footprint Resistors_SMD:R_0805 -> Resistors_SMD:R_0805_HandSoldering
- R8: value 100k -> 500; footprint Resistors_SMD:R_0805 -> Resistors_SMD:R_0805_HandSoldering
- SW1: renamed from WifiSw1; value SW_PUSH -> WifiReset; footprint Buttons_Switches_SMD:SW_SPST_EVQPE1 -> ASKicadLib:SW_PUSH_AS
- SW2: value SW_PUSH -> Flash; footprint Buttons_Switches_SMD:SW_SPST_EVQPE1 -> Pin_Headers:Pin_Header_Straight_1x02_Pitch2.54mm
- U3: footprint TO_SOT_Packages_SMD:SOT-23-5 -> TO_SOT_Packages_SMD:SOT-23-5_HandSoldering
Connections:
- net GND: now also FB1.2; no longer C4.1, C9.1, P3.1 (P1), R4.1, R9.2, U4.3 (Vin-), U4.4 (VSS)
- net VCC: now also C10.2, C4.1, C5.2, R5.2, R6.1, U3.5 (V+), U4.1 (Vref), U4.8 (VDD); no longer FB1.2
- net at U4.2 (Vin+): now also R8.1, C8.1; no longer C7.2
- net at P3.2 (P2), R5.1: now also C7.1; no longer C3.2
- net at R4.2, R7.1, U3.4 (IN-): now also C3.2; no longer R8.1
- net at C9.2, R6.2, R9.1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: no longer C3.1
- net at R8.2, U3.1 (OUT): now also C3.1, R4.1
- net GNDA: now reaches U3.2 (V-)
- net GNDA: now also C4.2, C9.1, FB1.1, P3.1 (P1), R9.2, U4.3 (Vin-), U4.4 (VSS), C8.2
- new net: C7.2, R7.2
Other:
- moved on the sheet: C9, FB1, P3, R5, R6, R7, R9, U3
