File: hardware/PCB/UsbSticka/03dev/03devOPAdual4layer.sch (KiCad schematic (older format))
At the start: 33 parts, among them P1 USB_B, P2 Debug, P3 MIC, SW2 SW_PUSH, U1 LM1117-3.3, U2 ESP-07v2, U3 OPA345, U4 MCP3201, U5 OPA345

Commit message: Dev08
Parts:
- removed P2: Debug, Socket_Strips:Socket_Strip_Straight_1x03, symbol CONN_01X03
- removed SW2: SW_PUSH, Buttons_Switches_SMD:SW_SPST_EVQPE1, symbol SW_PUSH
- added C12: 10uF, Capacitors_SMD:C_0805_HandSoldering, symbol C
- added C8: 0,1uF, Capacitors_SMD:C_0805_HandSoldering, symbol C
- C1, C11, C2, C3, C4, C5, C7, C9: footprint Capacitors_SMD:C_0805 -> Capacitors_SMD:C_0805_HandSoldering
- C10: value 0,1 -> 1.0uF; footprint Capacitors_SMD:C_0805 -> Capacitors_SMD:C_0805_HandSoldering
- C6: value 0,1uF -> 10uF; footprint Capacitors_SMD:C_0805 -> Capacitors_SMD:C_0805_HandSoldering
- R1, R10, R11, R12, R2, R3, R4, R5, R6, R7, R8, R9: footprint Resistors_SMD:R_0805 -> Resistors_SMD:R_0805_HandSoldering
- U3, U5: footprint TO_SOT_Packages_SMD:SOT-23-5 -> TO_SOT_Packages_SMD:SOT-23-5_HandSoldering
- U4: footprint Power_Integrations:PDIP-8 -> Housings_SOIC:SOIC-8_3.9x4.9mm_Pitch1.27mm
- WifiSw1: footprint Buttons_Switches_SMD:SW_SPST_EVQPE1 -> ASKicadLib:SW_PUSH_AS
Connections:
- net GND: now also C6.1, FB1.1, R3.1; no longer C10.1, C4.1, C6.2, C9.1, P3.1 (P1), R3.2, R4.1, R9.2, U4.3 (Vin-), U4.4 (VSS), U5.2 (V-)
- net SS: now also R3.2; no longer R3.1
- net VCC: now also C10.2, C5.2, C6.2, R5.2, R6.1, R7.2, U3.5 (V+), U4.1 (Vref), U4.8 (VDD), C12.2, C8.1; no longer C6.1, FB1.2
- new net GNDA: C10.1, C12.1, C4.1, C8.2, C9.1, FB1.2, P3.1 (P1), R4.1, R9.2, U4.3 (Vin-), U4.4 (VSS), U5.2 (V-)
- no-connect marks 8 -> 9
Other:
- moved on the sheet: C10, FB1, R3
